File: ad.kicad_sch (KiCad schematic)
At the start: 5 parts, among them U6 TAC5242

Commit message: modified:   MCU.kicad_sch 	modified:   PSU.kicad_sch 	modified:   ProjectY.kicad_pro 	modified:   ProjectY.kicad_sch 	modified:   ad.kicad_sch 	modified:   audio.kicad_sch
Parts:
- removed C13, C25: 10u, symbol Device:C
- removed C23, C26: 1u, symbol Device:C
- removed U6: TAC5242, Package_DFN_QFN:VQFN-24-1EP_4x4mm_P0.5mm_EP2.5x2.5mm_ThermalVias, symbol User:TAC5242
