File: ProjectY.kicad_sch (KiCad schematic)
At the start: 8 parts, among them J2 NRJ6HF, J3 9V, J4 NRJ6HF, J5 NRJ6HF, J6 AudioJack3, J7 AudioJack3, P1 USB_C

Commit message: modified:   MCU.kicad_sch 	modified:   PSU.kicad_sch 	modified:   ProjectY.kicad_pro 	modified:   ProjectY.kicad_sch 	modified:   ad.kicad_sch 	modified:   audio.kicad_sch
Other:
- removed sheet Audio Codec
- sheet Analog Audio ports: added +7VA, 3.3V, 3.3VA, GP0, I2S_CK, I2S_SDI, I2S_SDO, I2S_WS; removed +8VA, -8VA, ADC_L+, ADC_L-, ADC_R+, ADC_R-, CTR_Drythrough, DAC_L+, DAC_L-, DAC_R+, DAC_R-
- sheet PSU ports: added +7VA; removed +8VA, -8VA
- moved on the sheet: J2, J4, J5

Commit message: modified:   MCU.kicad_sch 	modified:   PSU.kicad_sch 	modified:   ProjectY.kicad_pro 	modified:   ProjectY.kicad_sch 	modified:   audio.kicad_sch 	modified:   fp-info-cache 	new file:   spdif.kicad_sch 	modified:   usbfilter.kicad_sch
Parts:
- removed J6, J7: AudioJack3, Connector_Audio:Jack_3.5mm_CUI_SJ-3523-SMT_Horizontal, symbol Connector_Audio:AudioJack3
- added J6: SPDIF_IN, symbol Connector:Conn_Coaxial
- added J7: SPDIF_OUT, symbol Connector:Conn_Coaxial
Connections:
- net PSU/+9V_return is gone; now on net GND: J3.1
- net GND: now also J6.2 (Ext), J7.2 (Ext)
- net USB-C filter/CC renamed PSU/CC
- net USB-C filter/D+ renamed PSU/D+
- net USB-C filter/D- renamed PSU/D-
- net USB-C filter/VBUS renamed PSU/VBUS
- net USB-C filter/VCONN renamed PSU/VCONN
Other:
- removed sheet USB-C filter
- added sheet SPDIF (spdif.kicad_sch)
- sheet DSP ports: added none; removed CTR_Drythrough
- sheet PSU ports: added CC, D+, D-, Dfiltered+, Dfiltered-, VBUS, VBUS_detect, VCONN; removed +9V_return
- moved on the sheet: J2, J3, J4, J5, P1

Commit message: asd
Parts:
- removed J2: NRJ6HF, Connector_Audio:Jack_6.35mm_Neutrik_NRJ6HF_Horizontal, symbol Connector_Audio:NRJ6HF
- removed J6: SPDIF_IN, symbol Connector:Conn_Coaxial
- removed N1: Housing, Enclosures:Hammond_1590BB, symbol Mechanical:Housing
- added J10, J6: NRJ6HF, Connector_Audio:Jack_6.35mm_Neutrik_NRJ6HF_Horizontal, symbol Connector_Audio:NRJ6HF
- added J2: Conn_ARM_JTAG_SWD_10, symbol Connector:Conn_ARM_JTAG_SWD_10
- added J8: Midi In, Connector_Audio:Jack_3.5mm_Lumberg_1503_07_Horizontal, symbol Connector_Audio:AudioJack3
- added J9: MIDI Out, Connector_Audio:Jack_3.5mm_Lumberg_1503_07_Horizontal, symbol Connector_Audio:AudioJack3
Connections:
- net GND: now also J10.RN, J10.S, J10.SN, J10.TN, J2.3 (GND), J2.5 (GND), J2.9 (GNDDetect), J6.RN, J6.S, J6.SN, J6.TN
- net DSP/SPDIF_OUT: now reaches J7.1 (In)
- net Analog Audio/Line_Output_L+ renamed Line_Output_L+
- net Analog Audio/Line_Output_L- renamed Line_Output_L-
- net Analog Audio/Line_Output_R+ renamed Line_Output_R+
- net Analog Audio/Line_Output_R- renamed Line_Output_R-
- new net DSP/SWCLK: J2.4 (SWCLK/TCK)
- new net DSP/SWDIO: J2.2 (SWDIO/TMS)
- new net DSP/SWO: J2.6 (SWO/TDO)
- new net DSP/VTREF: J2.1 (VTref)
- new net DSP/~{RESET}: J2.10 (~{RESET})
- new net IN_L+: J6.T
- new net IN_L-: J6.R
- new net IN_R+: J10.T
- new net IN_R-: J10.R
- new net MIDI + UI/MIDI IN Shield: J8.S
- new net MIDI + UI/MIDI OUT Shield: J9.S
- new net MIDI + UI/MIDI Out Sink: J9.T
- new net MIDI + UI/MIDI Out Source: J9.R
- new net MIDI + UI/Midi In Sink: J8.T
- new net MIDI + UI/Midi In Source: J8.R
- no-connect marks 6 -> 7
Other:
- sheet SPDIF renamed MIDI + UI
- sheet Analog Audio ports: added +3.3V, +3.3VA, +4.5V, -4.5V, IN_L+, IN_L-, IN_R+, IN_R-, ~{Dry_Through}, ~{Hi-Z}; removed +7VA, 3.3V, 3.3VA, Guitar_IN_L, Guitar_IN_R
- sheet DSP ports: added +3.3V, 2.5V_VREF, Footswitch_1, Footswitch_2, MIDI_UART0_RX, MIDI_UART0_TX, Potentiometer_1, Potentiometer_2, Potentiometer_3, Potentiometer_4, Potentiometer_5, Potentiometer_6, SPDIF_OUT, SWCLK, SWDIO, SWO, Switch_1A, Switch_1B, Switch_2A, Switch_2B, VTREF, ~{Dry_Through}, ~{Hi-Z}, ~{RESET}; removed 3V3
- sheet MIDI + UI ports: added +2.5VA, +3.3V, Footswitch_1, Footswitch_2, MIDI IN Shield, MIDI OUT Shield, MIDI Out Sink, MIDI Out Source, Midi In Sink, Midi In Source, Potentiometer_1, Potentiometer_2, Potentiometer_3, Potentiometer_4, Potentiometer_5, Potentiometer_6, Switch_1A, Switch_1B, Switch_2A, Switch_2B, UART0_RX, UART0_TX; removed none
- sheet PSU ports: added +2.5VA, +4.5V, -4.5V, PSU_ST, VBUS_DETECT; removed +7VA, VBUS_detect
- note added: "In L"
- note added: "In R"
- note added: "Potentiometers Switches Footswitches LEDs"
- moved on the sheet: J3, J4, J5, J7, P1

Commit message: git test
Other:
- note added: "GIT TEST"
Changed lines of the file:
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@@
+		)
+	)
+	(text "GIT TEST\n"
+		(exclude_from_sim no)
+		(at 102.87 44.958 0)
+		(effects
+			(font
+				(size 25.4 25.4)
+			)
 		)
 	)

Commit message: added decoupling for DSP
Other:
- sheet Analog Audio ports: added none; removed ~{Dry_Through}, ~{Hi-Z}
- sheet DSP ports: added none; removed ~{Dry_Through}, ~{Hi-Z}
- sheet MIDI + UI ports: added +3.3VA2; removed none
- sheet PSU ports: added 3.3VA2; removed none
- note removed: "GIT TEST"
Changed lines of the file:
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@@
 		)
 	)
-	(text "GIT TEST\n"
-		(exclude_from_sim no)
-		(at 102.87 44.958 0)
-		(effects
-			(font
-				(size 25.4 25.4)
-			)
-		)
-	)
 	(junction
 		(at 83.82 251.46)
@@
 	)
 	(junction
-		(at 83.82 224.79)
+		(at 185.42 115.57)
 		(diameter 0)
 		(color 0 0 0 0)
 	)
 	(junction
-		(at 83.82 227.33)
+		(at 83.82 224.79)
 		(diameter 0)
 		(color 0 0 0 0)
 	)
 	(junction
-		(at 185.42 111.76)
+		(at 83.82 227.33)
 		(diameter 0)
 		(color 0 0 0 0)
@@
 	(wire
 		(pts
+			(xy 130.81 113.03) (xy 179.07 113.03)
+		)
+		(stroke
+			(width 0)
+			(type default)
+		)
+	)
+	(wire
+		(pts
 			(xy 208.28 71.12) (xy 203.2 71.12)
 		)
@@
 	(wire
 		(pts
+			(xy 179.07 90.17) (xy 208.28 90.17)
+		)
+		(stroke
+			(width 0)
+			(type default)
+		)
+	)
+	(wire
+		(pts
 			(xy 269.24 193.04) (xy 242.57 193.04)
 		)
@@
 	(wire
 		(pts
-			(xy 208.28 90.17) (xy 185.42 90.17)
+			(xy 208.28 92.71) (xy 185.42 92.71)
 		)
 		(stroke
@@
 	(wire
 		(pts
-			(xy 185.42 90.17) (xy 185.42 111.76)
+			(xy 179.07 113.03) (xy 179.07 90.17)
 		)
 		(stroke
@@
 	(wire
 		(pts
-			(xy 130.81 111.76) (xy 185.42 111.76)
+			(xy 130.81 115.57) (xy 185.42 115.57)
 		)
 		(stroke
@@
 	(wire
 		(pts
+			(xy 185.42 92.71) (xy 185.42 115.57)
+		)
+		(stroke
+			(width 0)
+			(type default)
+		)
+	)
+	(wire
+		(pts
 			(xy 130.81 143.51) (xy 180.34 143.51)
 		)
@@
 	(wire
 		(pts
-			(xy 185.42 111.76) (xy 208.28 111.76)
+			(xy 185.42 115.57) (xy 208.28 115.57)
 		)
 		(stroke
@@
 			)
 		)
-		(pin "~{Dry_Through}" input
-			(at 223.52 158.75 90)
-			(effects
-				(font
-					(size 1.27 1.27)
-				)
-				(justify right)
-			)
-		)
-		(pin "~{Hi-Z}" input
-			(at 220.98 158.75 90)
-			(effects
-				(font
-					(size 1.27 1.27)
-				)
-				(justify right)
-			)
-		)
 		(instances
 			(project "ProjectY"
@@
 		)
 		(pin "+2.5VA" input
-			(at 208.28 90.17 180)
+			(at 208.28 92.71 180)
 			(effects
 				(font
@@
 			)
 		)
+		(pin "+3.3VA2" input
+			(at 208.28 90.17 180)
+			(effects
+				(font
+					(size 1.27 1.27)
+				)
+				(justify left)
+			)
+		)
 		(instances
 			(project "ProjectY"
@@
 		)
 		(pin "2.5V_VREF" input
-			(at 208.28 111.76 180)
-			(effects
-				(font
-					(size 1.27 1.27)
-				)
-				(justify left)
-			)
-		)
-		(pin "~{Dry_Through}" input
-			(at 223.52 143.51 270)
-			(effects
-				(font
-					(size 1.27 1.27)
-				)
-				(justify left)
-			)
-		)
-		(pin "~{Hi-Z}" input
-			(at 220.98 143.51 270)
+			(at 208.28 115.57 180)
 			(effects
 				(font
@@
 		)
 		(pin "+2.5VA" input
-			(at 130.81 111.76 0)
+			(at 130.81 115.57 0)
+			(effects
+				(font
+					(size 1.27 1.27)
+				)
+				(justify right)
+			)
+		)
+		(pin "3.3VA2" input
+			(at 130.81 113.03 0)
 			(effects
 				(font

Commit message: commit
Other:
- sheet DSP ports: added none; removed MIDI_UART0_TX
- sheet MIDI + UI ports: added none; removed UART0_TX
Changed lines of the file:
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@@
-	(wire
-		(pts
-			(xy 224.79 97.79) (xy 224.79 107.95)
-		)
-		(stroke
-			(width 0)
-			(type default)
-		)
-	)
 	(wire
 		(pts
@@
 			)
 		)
-		(pin "UART0_TX" input
-			(at 224.79 97.79 270)
-			(effects
-				(font
-					(size 1.27 1.27)
-				)
-				(justify left)
-			)
-		)
 		(pin "Midi In Source" input
 			(at 208.28 71.12 180)
@@
 			(effects
 				(font
-					(size 1.27 1.27)
-				)
-				(justify right)
-			)
-		)
-		(pin "MIDI_UART0_TX" input
-			(at 224.79 107.95 90)
-			(effects
-				(font

Commit message: started the layout process
Parts:
- removed J9: MIDI Out, Connector_Audio:Jack_3.5mm_Lumberg_1503_07_Horizontal, symbol Connector_Audio:AudioJack3
- removed P1: USB_C, Connector_USB:USB_C_Receptacle_GCT_USB4110, symbol Connector:USB_C_Plug_USB2.0
- added J9: USB_C_Receptacle_USB2.0_14P, Connector_USB:USB_C_Receptacle_GCT_USB4110, symbol Connector:USB_C_Receptacle_USB2.0_14P
- J2: footprint (none) -> Connector_PinHeader_1.27mm:PinHeader_2x05_P1.27mm_Vertical_SMD
Connections:
- net GND: now also J9.A1 (GND), J9.A12 (GND), J9.B1 (GND), J9.B12 (GND), J9.S1 (SHIELD)
- net PSU/CC: now also J9.A5 (CC1)
- net PSU/D+: now also J9.A6 (D+), J9.B6 (D+)
- net PSU/D-: now also J9.A7 (D-), J9.B7 (D-)
- net PSU/VBUS: now also J9.A4 (VBUS), J9.A9 (VBUS), J9.B4 (VBUS), J9.B9 (VBUS)
- net PSU/VCONN: now also J9.B5 (CC2)
Changed lines of the file:
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@@
+	)
+	(junction
+		(at 100.33 144.78)
+		(diameter 0)
+		(color 0 0 0 0)
 	)
 	(junction
@@
 		(color 255 0 0 1)
 	)
+	(junction
+		(at 100.33 149.86)
+		(diameter 0)
+		(color 0 0 0 0)
+	)
 	(no_connect
 		(at 308.61 125.73)
@@
 	(wire
 		(pts
+			(xy 100.33 147.32) (xy 100.33 144.78)
+		)
+		(stroke
+			(width 0)
+			(type default)
+		)
+	)
+	(wire
+		(pts
 			(xy 283.21 170.18) (xy 271.78 170.18)
 		)
@@
 	(wire
 		(pts
-			(xy 262.89 71.12) (xy 281.94 71.12)
-		)
-		(stroke
-			(width 0)
-			(type default)
-		)
-	)
-	(wire
-		(pts
 			(xy 171.45 147.32) (xy 171.45 170.18)
 		)
@@
 	(wire
 		(pts
+			(xy 100.33 144.78) (xy 105.41 144.78)
+		)
+		(stroke
+			(width 0)
+			(type default)
+		)
+	)
+	(wire
+		(pts
 			(xy 233.68 143.51) (xy 233.68 158.75)
 		)
@@
 	(wire
 		(pts
-			(xy 262.89 73.66) (xy 281.94 73.66)
-		)
-		(stroke
-			(width 0)
-			(type default)
-		)
-	)
-	(wire
-		(pts
 			(xy 182.88 193.04) (xy 208.28 193.04)
 		)
@@
 	(wire
 		(pts
-			(xy 262.89 68.58) (xy 281.94 68.58)
-		)
-		(stroke
-			(width 0)
-			(type default)
-		)
-	)
-	(wire
-		(pts
 			(xy 208.28 95.25) (xy 196.85 95.25)
 		)
@@
 	(wire
 		(pts
-			(xy 100.33 144.78) (xy 105.41 144.78)
-		)
-		(stroke
-			(width 0)
-			(type default)
-		)
-	)
-	(wire
-		(pts
 			(xy 83.82 241.3) (xy 83.82 246.38)
 		)
@@
 		(pts
 			(xy 130.81 147.32) (xy 171.45 147.32)
+		)
+		(stroke
+			(width 0)
+			(type default)
+		)
+	)
+	(wire
+		(pts
+			(xy 100.33 149.86) (xy 100.33 152.4)
 		)
 		(stroke
@@
 	)
 	(symbol
+		(lib_id "Connector:USB_C_Receptacle_USB2.0_14P")
+		(at 85.09 147.32 0)
+		(unit 1)
+		(exclude_from_sim no)
+		(in_bom yes)
+		(on_board yes)
+		(dnp no)
+		(fields_autoplaced yes)
+		(property "Reference" "J9"
+			(at 85.09 124.46 0)
+			(effects
+				(font
+					(size 1.27 1.27)
+				)
+			)
+		)
+		(property "Value" "USB_C_Receptacle_USB2.0_14P"
+			(at 85.09 127 0)
+			(effects
+				(font
+					(size 1.27 1.27)
+				)
+			)
+		)
+		(property "Footprint" "Connector_USB:USB_C_Receptacle_GCT_USB4110"
+			(at 88.9 147.32 0)
+			(effects
+				(font
+					(size 1.27 1.27)
+				)
+				(hide yes)
+			)
+		)
+		(property "Datasheet" "https://www.usb.org/sites/default/files/documents/usb_type-c.zip"
+			(at 88.9 147.32 0)
+			(effects
+				(font
+					(size 1.27 1.27)
+				)
+				(hide yes)
+			)
+		)
+		(property "Description" "USB 2.0-only 14P Type-C Receptacle connector"
+			(at 85.09 147.32 0)
+			(effects
+				(font
+					(size 1.27 1.27)
+				)
+				(hide yes)
+			)
+		)
+		(pin "B5"
+		)
+		(pin "A5"
+		)
+		(pin "A1"
+		)
+		(pin "A9"
+		)
+		(pin "A4"
+		)
+		(pin "A12"
+		)
+		(pin "B1"
+		)
+		(pin "B12"
+		)
+		(pin "B4"
+		)
+		(pin "S1"
+		)
+		(pin "B9"
+		)
+		(pin "A6"
+		)
+		(pin "A7"
+		)
+		(pin "B7"
+		)
+		(pin "B6"
+		)
+		(instances
+			(project ""
+				(path "/6b669608-d244-47fa-b233-c11102b937f7"
+					(reference "J9")
+					(unit 1)
+				)
+			)
+		)
+	)
+	(symbol
 		(lib_id "power:GND")
 		(at 83.82 229.87 0)
@@
 				(path "/6b669608-d244-47fa-b233-c11102b937f7"
 					(reference "J3")
-					(unit 1)
-				)
-			)
-		)
-	)
-	(symbol
-		(lib_id "Connector_Audio:AudioJack3")
-		(at 287.02 71.12 180)
-		(unit 1)
-		(exclude_from_sim no)
-		(in_bom yes)
-		(on_board yes)
-		(dnp no)
-		(property "Reference" "J9"
-			(at 287.02 78.74 0)
-			(effects
-				(font
-					(size 1.27 1.27)
-				)
-			)
-		)
-		(property "Value" "MIDI Out"
-			(at 287.02 76.2 0)
-			(effects
-				(font
-					(size 1.27 1.27)
-				)
-			)
-		)
-		(property "Footprint" "Connector_Audio:Jack_3.5mm_Lumberg_1503_07_Horizontal"
-			(at 287.02 71.12 0)
-			(effects
-				(font
-					(size 1.27 1.27)
-				)
-				(hide yes)
-			)
-		)
-		(property "Datasheet" "~"
-			(at 287.02 71.12 0)
-			(effects
-				(font
-					(size 1.27 1.27)
-				)
-				(hide yes)
-			)
-		)
-		(property "Description" "Audio Jack, 3 Poles (Stereo / TRS)"
-			(at 287.02 71.12 0)
-			(effects
-				(font
-					(size 1.27 1.27)
-				)
-				(hide yes)
-			)
-		)
-		(pin "R"
-		)
-		(pin "S"
-		)
-		(pin "T"
-		)
-		(instances
-			(project "ProjectY"
-				(path "/6b669608-d244-47fa-b233-c11102b937f7"
-					(reference "J9")
-					(unit 1)
-				)
-			)
-		)
-	)
-	(symbol
-		(lib_id "Connector:USB_C_Plug_USB2.0")
-		(at 85.09 147.32 0)
-		(unit 1)
-		(exclude_from_sim no)
-		(in_bom yes)
-		(on_board yes)
-		(dnp no)
-		(property "Reference" "P1"
-			(at 85.852 124.968 0)
-			(effects
-				(font
-					(size 1.27 1.27)
-				)
-				(justify right)
-			)
-		)
-		(property "Value" "USB_C"
-			(at 88.138 127.508 0)
-			(effects
-				(font
-					(size 1.27 1.27)
-				)
-				(justify right)
-			)
-		)
-		(property "Footprint" "Connector_USB:USB_C_Receptacle_GCT_USB4110"
-			(at 88.9 147.32 0)
-			(effects
-				(font
-					(size 1.27 1.27)
-				)
-				(hide yes)
-			)
-		)
-		(property "Datasheet" "https://www.usb.org/sites/default/files/documents/usb_type-c.zip"
-			(at 88.9 147.32 0)
-			(effects
-				(font
-					(size 1.27 1.27)
-				)
-				(hide yes)
-			)
-		)
-		(property "Description" "USB 2.0-only Type-C Plug connector"
-			(at 85.09 147.32 0)
-			(effects
-				(font
-					(size 1.27 1.27)
-				)
-				(hide yes)
-			)
-		)
-		(pin "A5"
-		)
-		(pin "A6"
-		)
-		(pin "B4"
-		)
-		(pin "A9"
-		)
-		(pin "B1"
-		)
-		(pin "S1"
-		)
-		(pin "A7"
-		)
-		(pin "A12"
-		)
-		(pin "B12"
-		)
-		(pin "A1"
-		)
-		(pin "B9"
-		)
-		(pin "B5"
-		)
-		(pin "A4"
-		)
-		(instances
-			(project "ProjectY"
-				(path "/6b669608-d244-47fa-b233-c11102b937f7"
-					(reference "P1")
 					(unit 1)
 				)
@@
 			)
 		)
-		(property "Footprint" ""
+		(property "Footprint" "Connector_PinHeader_1.27mm:PinHeader_2x05_P1.27mm_Vertical_SMD"
 			(at 321.31 120.65 0)
 			(effects
@@
 	(symbol
 		(lib_id "power:GND")
-		(at 77.47 170.18 0)
+		(at 85.09 170.18 0)
 		(unit 1)
 		(exclude_from_sim no)
@@
 		(dnp no)
 		(fields_autoplaced yes)
-		(property "Reference" "#PWR039"
-			(at 77.47 176.53 0)
+		(property "Reference" "#PWR038"
+			(at 85.09 176.53 0)
 			(effects
 				(font
@@
 		)
 		(property "Value" "GND"
-			(at 77.47 175.26 0)
+			(at 85.09 175.26 0)
 			(effects
 				(font
@@
 		)
 		(property "Footprint" ""
-			(at 77.47 170.18 0)
+			(at 85.09 170.18 0)
 			(effects
 				(font
@@
 		)
 		(property "Datasheet" ""
-			(at 77.47 170.18 0)
+			(at 85.09 170.18 0)
 			(effects
 				(font
@@
 		)
 		(property "Description" "Power symbol creates a global label with name \"GND\" , ground"
-			(at 77.47 170.18 0)
+			(at 85.09 170.18 0)
 			(effects
 				(font
@@
 			(project "ProjectY"
 				(path "/6b669608-d244-47fa-b233-c11102b937f7"
-					(reference "#PWR039")
+					(reference "#PWR038")
 					(unit 1)
 				)
@@
 	(symbol
 		(lib_id "power:GND")
-		(at 85.09 170.18 0)
+		(at 77.47 170.18 0)
 		(unit 1)
 		(exclude_from_sim no)
@@
 		(dnp no)
 		(fields_autoplaced yes)
-		(property "Reference" "#PWR038"
-			(at 85.09 176.53 0)
+		(property "Reference" "#PWR039"
+			(at 77.47 176.53 0)
 			(effects
 				(font
@@
 		)
 		(property "Value" "GND"
-			(at 85.09 175.26 0)
+			(at 77.47 175.26 0)
 			(effects
 				(font
@@
 		)
 		(property "Footprint" ""
-			(at 85.09 170.18 0)
+			(at 77.47 170.18 0)
 			(effects
 				(font
@@
 		)
 		(property "Datasheet" ""
-			(at 85.09 170.18 0)
+			(at 77.47 170.18 0)
 			(effects
 				(font
@@
 		)
 		(property "Description" "Power symbol creates a global label with name \"GND\" , ground"
-			(at 85.09 170.18 0)
+			(at 77.47 170.18 0)
 			(effects
 				(font
@@
 			(project "ProjectY"
 				(path "/6b669608-d244-47fa-b233-c11102b937f7"
-					(reference "#PWR038")
+					(reference "#PWR039")
 					(unit 1)
 				)

Commit message: lot of changes
Parts:
- removed J10, J4: NRJ6HF, Connector_Audio:Jack_6.35mm_Neutrik_NRJ6HF_Horizontal, symbol Connector_Audio:NRJ6HF
- removed J7: SPDIF_OUT, symbol Connector:Conn_Coaxial
- removed J8: Midi In, Connector_Audio:Jack_3.5mm_Lumberg_1503_07_Horizontal, symbol Connector_Audio:AudioJack3
- added J7: MIDI In, User:Jack_6.35mm_Neutrik_NRJ6HF_Horizontal, symbol Connector_Audio:NRJ6HF
- J3: footprint Connector_BarrelJack:BarrelJack_GCT_DCJ200-10-A_Horizontal -> User:BarrelJack_GCT_DCJ200-10-A_Horizontal
- J5: value NRJ6HF -> Out; footprint Connector_Audio:Jack_6.35mm_Neutrik_NRJ6HF_Horizontal -> User:Jack_6.35mm_Neutrik_NRJ6HF_Horizontal; PN (none) -> NRJ6HF
- J6: value NRJ6HF -> IN; footprint Connector_Audio:Jack_6.35mm_Neutrik_NRJ6HF_Horizontal -> User:Jack_6.35mm_Neutrik_NRJ6HF_Horizontal; PN (none) -> NRJ6HF
- J9: footprint Connector_USB:USB_C_Receptacle_GCT_USB4110 -> User:USB_C_Receptacle_GCT_USB4110
Connections:
- net PSU/D+ is gone; now on net DSP/D+: J9.A6 (D+), J9.B6 (D+)
- net PSU/D- is gone; now on net DSP/D-: J9.A7 (D-), J9.B7 (D-)
- net IN_L+ renamed Analog Audio/IN_L
- net IN_L- renamed Analog Audio/IN_R
- net Line_Output_L+ renamed Analog Audio/Line_Output_L
- net Line_Output_L- renamed Analog Audio/Line_Output_R
- net PSU/CC renamed DSP/CC
- net PSU/VBUS renamed DSP/VBUS
- net PSU/VCONN renamed DSP/VCONN
- new net DSP/MIDI IN Shield: J7.S
- new net DSP/Midi In Sink: J7.T
- new net DSP/Midi In Source: J7.R
Other:
- sheet Analog Audio ports: added +V_OPA, -V_OPA, IN_L, IN_R, Line_Output_L, Line_Output_R; removed +3.3VA, +4.5V, -4.5V, IN_L+, IN_L-, IN_R+, IN_R-, Line_Output_L+, Line_Output_L-, Line_Output_R+, Line_Output_R-
- sheet DSP ports: added +2.5VA, CC, MIDI IN Shield, Midi In Sink, Midi In Source, VBUS, VCONN; removed 2.5V_VREF, MIDI_UART0_RX, SPDIF_OUT, VBUS_detect
- sheet MIDI + UI ports: added none; removed +3.3VA2, MIDI IN Shield, MIDI OUT Shield, MIDI Out Sink, MIDI Out Source, Midi In Sink, Midi In Source, UART0_RX
- sheet PSU ports: added +V_OPA, -V_OPA; removed +3.3VA, +4.5V, -4.5V, 3.3VA2, CC, D+, D-, Dfiltered+, Dfiltered-, PSU_ST, VBUS, VBUS_DETECT, VCONN
- note removed: "In L"
- note removed: "In R"
- moved on the sheet: J5, J6, J9
