File: ProjectY.kicad_sch (KiCad schematic)
At the start: 6 parts, among them J2 Conn_ARM_JTAG_SWD_10, J3 9V, J5 Out, J6 IN, J7 MIDI In, J9 USB_C_Receptacle_USB2.0_14P

Commit message: last stm32h7 version
Parts:
- added J15, J16: 009155002852006, User:KYO_009155002852006, symbol Thunderscope_Rev5:CONN SPRING 2 PIN
Connections:
- net DSP/MIDI IN Shield: now also J7.RN, J7.SN, J7.TN
- net GND: now also J15.1, J15.2, J16.1, J16.2
- no-connect marks 7 -> 4
