File: MCU.kicad_sch (KiCad schematic)
At the start: 22 parts, among them J1 Conn_ARM_JTAG_SWD_10, U1 MT48LC16M16A2P, U2 W25Q128JVS, U3 STM32H743ZGTx

Commit message: modified:   MCU.kicad_sch 	modified:   PSU.kicad_sch 	modified:   ProjectY.kicad_pro 	modified:   ProjectY.kicad_sch 	modified:   ad.kicad_sch 	modified:   audio.kicad_sch
Parts:
- removed C1, C11, C12, C14, C15, C16, C17, C18, C19, C2, C20, C3, C4, C5, C6, C7, C9: 2.2u, symbol Device:C
- added C12, C14, C25, C26, C41, C42, C48, C59, C60, C61, C62, C63, C64, C65, C66, C67, C68, C70: 2.2uF, PCM_JLCPCB:C_0402, symbol PCM_JLCPCB-Capacitors:0402,2.2uF
Connections:
- net 3V3: now also C26.1, C41.1, C42.1, C48.1, C59.1, C60.1, C61.1, C62.1, C63.1, C64.1, C65.1, C66.1, C67.1, C68.1, C70.1
- net GND: now also C14.2, C25.2, C26.2, C41.2, C42.2, C48.2, C59.2, C60.2, C61.2, C62.2, C63.2, C64.2, C65.2, C66.2, C67.2, C68.2, C70.2
- net at U3.106 (VCAP): now also C14.1
- net at U3.71 (VCAP): now also C25.1

Commit message: modified:   MCU.kicad_sch 	modified:   PSU.kicad_sch 	modified:   ProjectY.kicad_pro 	modified:   ProjectY.kicad_sch 	modified:   audio.kicad_sch 	modified:   fp-info-cache 	new file:   spdif.kicad_sch 	modified:   usbfilter.kicad_sch
Parts:
- removed C12: 2.2uF, PCM_JLCPCB:C_0402, symbol PCM_JLCPCB-Capacitors:0402,2.2uF
Changed lines of the file:
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@@
-	(symbol
-		(lib_id "PCM_JLCPCB-Capacitors:0402,2.2uF")
-		(at 83.82 193.04 0)
-		(unit 1)
-		(exclude_from_sim no)
-		(in_bom yes)
-		(on_board yes)
-		(dnp no)
-		(fields_autoplaced yes)
-		(property "Reference" "C12"
-			(at 86.36 190.4999 0)
-			(effects
-				(font
-					(size 1.27 1.27)
-				)
-				(justify left)
-			)
-		)
-		(property "Value" "2.2uF"
-			(at 86.36 193.04 0)
-			(effects
-				(font
-					(size 0.8 0.8)
-				)
-				(justify left)
-			)
-		)
-		(property "Footprint" "PCM_JLCPCB:C_0402"
-			(at 82.042 193.04 90)
-			(effects
-				(font
-					(size 1.27 1.27)
-				)
-				(hide yes)
-			)
-		)
-		(property "Datasheet" "https://www.lcsc.com/datasheet/lcsc_datasheet_2304140030_Samsung-Electro-Mechanics-CL05A225MQ5NSNC_C12530.pdf"
-			(at 83.82 193.04 0)
-			(effects
-				(font
-					(size 1.27 1.27)
-				)
-				(hide yes)
-			)
-		)
-		(property "Description" "6.3V 2.2uF X5R ±20% 0402 Multilayer Ceramic Capacitors MLCC - SMD/SMT ROHS"
-			(at 83.82 193.04 0)
-			(effects
-				(font
-					(size 1.27 1.27)
-				)
-				(hide yes)
-			)
-		)
-		(property "LCSC" "C12530"
-			(at 83.82 193.04 0)
-			(effects
-				(font
-					(size 1.27 1.27)
-				)
-				(hide yes)
-			)
-		)
-		(property "Stock" "4665427"
-			(at 83.82 193.04 0)
-			(effects
-				(font
-					(size 1.27 1.27)
-				)
-				(hide yes)
-			)
-		)
-		(property "Price" "0.006USD"
-			(at 83.82 193.04 0)
-			(effects
-				(font
-					(size 1.27 1.27)
-				)
-				(hide yes)
-			)
-		)
-		(property "Process" "SMT"
-			(at 83.82 193.04 0)
-			(effects
-				(font
-					(size 1.27 1.27)
-				)
-				(hide yes)
-			)
-		)
-		(property "Minimum Qty" "20"
-			(at 83.82 193.04 0)
-			(effects
-				(font
-					(size 1.27 1.27)
-				)
-				(hide yes)
-			)
-		)
-		(property "Attrition Qty" "10"
-			(at 83.82 193.04 0)
-			(effects
-				(font
-					(size 1.27 1.27)
-				)
-				(hide yes)
-			)
-		)
-		(property "Class" "Basic Component"
-			(at 83.82 193.04 0)
-			(effects
-				(font
-					(size 1.27 1.27)
-				)
-				(hide yes)
-			)
-		)
-		(property "Category" "Capacitors,Multilayer Ceramic Capacitors MLCC - SMD/SMT"
-			(at 83.82 193.04 0)
-			(effects
-				(font
-					(size 1.27 1.27)
-				)
-				(hide yes)
-			)
-		)
-		(property "Manufacturer" "Samsung Electro-Mechanics"
-			(at 83.82 193.04 0)
-			(effects
-				(font
-					(size 1.27 1.27)
-				)
-				(hide yes)
-			)
-		)
-		(property "Part" "CL05A225MQ5NSNC"
-			(at 83.82 193.04 0)
-			(effects
-				(font
-					(size 1.27 1.27)
-				)
-				(hide yes)
-			)
-		)
-		(property "Voltage Rated" "6.3V"
-			(at 86.36 195.58 0)
-			(effects
-				(font
-					(size 0.8 0.8)
-				)
-				(justify left)
-			)
-		)
-		(property "Tolerance" "±20%"
-			(at 83.82 193.04 0)
-			(effects
-				(font
-					(size 1.27 1.27)
-				)
-				(hide yes)
-			)
-		)
-		(property "Capacitance" "2.2uF"
-			(at 83.82 193.04 0)
-			(effects
-				(font
-					(size 1.27 1.27)
-				)
-				(hide yes)
-			)
-		)
-		(property "Temperature Coefficient" "X5R"
-			(at 83.82 193.04 0)
-			(effects
-				(font
-					(size 1.27 1.27)
-				)
-				(hide yes)
-			)
-		)
-		(pin "2"
-		)
-		(pin "1"
-		)
-		(instances
-			(project ""
-				(path "/6b669608-d244-47fa-b233-c11102b937f7/942daa49-72f6-4fca-bb5b-9cd809da0775"
-					(reference "C12")
-					(unit 1)
-				)
-			)
-		)
-	)
 	(symbol
 		(lib_id "PCM_JLCPCB-Capacitors:0402,2.2uF")

Commit message: asd
Parts:
- removed C10: 100n, symbol Device:C_Small
- removed C14, C25, C26, C41, C42, C48, C59, C60, C61, C62, C63, C64, C65, C66, C67, C68, C70: 2.2uF, PCM_JLCPCB:C_0402, symbol PCM_JLCPCB-Capacitors:0402,2.2uF
- removed J1: Conn_ARM_JTAG_SWD_10, symbol Connector:Conn_ARM_JTAG_SWD_10
- removed U3: STM32H743ZGTx, Package_QFP:LQFP-144_20x20mm_P0.5mm, symbol MCU_ST_STM32H7:STM32H743ZGTx
- added C10: 100nF, PCM_JLCPCB:C_0402, symbol PCM_JLCPCB-Capacitors:0402,100nF
- added R1: 0Ω, PCM_JLCPCB:R_0402, symbol PCM_JLCPCB-Resistors:0402,0Ω
- added R15, R19: 1kΩ, PCM_JLCPCB:R_0402, symbol PCM_JLCPCB-Resistors:0402,1kΩ
- added U18: STM32H7R7I8Tx, Package_QFP:LQFP-176_24x24mm_P0.5mm, symbol MCU_ST_STM32H7:STM32H7R7I8Tx
- added U3: FM24CL64B, Package_SO:SOIC-8_3.9x4.9mm_P1.27mm, symbol Memory_NVRAM:FM24C64B
- added Y1: ASDLJ-E-49.152MHZ-L-R-T, Oscillator:Oscillator_SMD_Abracon_ASDMB-4Pin_2.5x2.0mm, symbol Oscillator:ASDMB-xxxMHz
- U1: value MT48LC16M16A2P -> W9825G6KH-6; LCSC (none) -> C97572
- U2: LCSC (none) -> C97521
Connections:
- net D+: now also U18.149 (PM11)
- net D-: now also U18.148 (PM12)
- net FLASH_CLK: now also U18.71 (PO4)
- net FLASH_QSPI0: now also U18.73 (PP0)
- net FLASH_QSPI1: now also U18.79 (PP1)
- net FLASH_QSPI2: now also U18.66 (PP2)
- net FLASH_QSPI3: now also U18.67 (PP3)
- net FLASH_~{CS}: now also U18.82 (PO0)
- net GND: now also C10.1, R1.1, U18.104 (VSS), U18.11 (VSS), U18.126 (VSS), U18.13 (VSSSMPS), U18.140 (VSS), U18.167 (VSS), U18.26 (VSS), U18.32 (VSSA), U18.40 (VSS), U18.52 (VSS), U18.6 (VSS), U18.60 (VSS), U18.64 (VSS), U18.68 (VSS), U18.74 (VSS), U18.80 (VSS), U18.90 (VSS), U18.94 (VSS), U18.98 (VSS), U3.1 (A0), U3.2 (A1), U3.3 (A2), U3.4 (VSS), Y1.2 (GND); no longer U1.12 (VSSQ), U1.28 (VSS), U1.41 (VSS), U1.46 (VSSQ), U1.52 (VSSQ), U1.54 (VSS), U1.6 (VSSQ), U2.4 (GND)
- net GPO: now also U18.48 (PB0)
- net I2S_CK: now also U18.43 (PA5)
- net I2S_SDI: now also U18.44 (PA6)
- net I2S_SDO: now also U18.45 (PA7)
- net I2S_WS: now also U18.42 (PA4)
- net RAM_A0: now also U18.29 (PC1)
- net RAM_A1: now also U18.30 (PC2)
- net RAM_A10: now also U18.160 (PF2)
- net RAM_A11: now also U18.161 (PF3)
- net RAM_A12: now also U18.55 (PE8)
- net RAM_A2: now also U18.31 (PC3)
- net RAM_A3: now also U18.46 (PC4)
- net RAM_A4: now also U18.54 (PE7)
- net RAM_A5: now also U18.47 (PC5)
- net RAM_A6: now also U18.132 (PD0)
- net RAM_A7: now also U18.133 (PD1)
- net RAM_A8: now also U18.158 (PF0)
- net RAM_A9: now also U18.159 (PF1)
- net RAM_BA0: now also U18.56 (PE9)
- net RAM_BA1: now also U18.57 (PE10)
- net RAM_CKE: now also U18.139 (PE15)
- net RAM_CLK: now also U18.101 (PN6)
- net RAM_D0: now also U18.103 (PN2)
- net RAM_D1: now also U18.109 (PN3)
- net RAM_D10: now also U18.84 (PB11)
- net RAM_D11: now also U18.83 (PB10)
- net RAM_D12: now also U18.7 (PE3)
- net RAM_D13: now also U18.8 (PE4)
- net RAM_D14: now also U18.9 (PE5)
- net RAM_D15: now also U18.10 (PE6)
- net RAM_D2: now also U18.96 (PN4)
- net RAM_D3: now also U18.97 (PN5)
- net RAM_D4: now also U18.95 (PN8)
- net RAM_D5: now also U18.102 (PN9)
- net RAM_D6: now also U18.106 (PN10)
- net RAM_D7: now also U18.108 (PN11)
- net RAM_D8: now also U18.86 (PB13)
- net RAM_D9: now also U18.85 (PB12)
- net RAM_DQMH: now also U18.28 (PC0)
- net RAM_DQML: now also U18.111 (PN1)
- net RAM_~{CAS}: now also U18.137 (PE13)
- net RAM_~{CS}: now also U18.138 (PE14)
- net RAM_~{RAS}: now also U18.136 (PE12)
- net RAM_~{WE}: now also U18.135 (PE11)
- net SWCLK: now also U18.123 (PA14(JTCK)
- net SWDIO: now also U18.122 (PA13(JTMS)
- net SWO: now also U18.163 (PB3(JTDO)
- net VBUS_detect: now also U18.150 (PM14)
- net ~{RESET}: now also C10.2, U18.25 (NRST)
- net 3V3 renamed +3.3V
- net +3.3V: now also R15.1, R19.1, U3.8 (VDD), Y1.1 (Standby), Y1.4 (VDD)
- new net: R1.2, U18.152 (BOOT0)
- new net: U18.23 (PH0), Y1.3 (Out)
- new net 2.5V_VREF: U18.34 (VREFP)
- new net FRAM_SCL: R19.2, U18.117 (PA8), U3.6 (SCL)
- new net FRAM_SDA: R15.2, U18.118 (PA9), U3.5 (SDA)
- new net FRAM_WP: U18.119 (PA10), U3.7 (WP)
- new net GNDD: U1.12 (VSSQ), U1.28 (VSS), U1.41 (VSS), U1.46 (VSSQ), U1.52 (VSSQ), U1.54 (VSS), U1.6 (VSSQ), U2.4 (GND)
- new net MIDI_UART0_RX: U18.120 (PA11)
- new net MIDI_UART0_TX: U18.121 (PA12)
- new net Potentiometer_1: U18.36 (PA0)
- new net Potentiometer_2: U18.37 (PA1)
- new net Potentiometer_3: U18.38 (PA2)
- new net Potentiometer_4: U18.39 (PA3)
- new net Potentiometer_5: U18.49 (PB1)
- new net Potentiometer_6: U18.53 (PF11)
- new net SPDIF_OUT: U18.50 (PB2)
- new net VTREF: U18.1 (VBAT), U18.116 (VDD), U18.12 (VDD), U18.128 (VDD), U18.141 (VDD), U18.157 (VDD), U18.169 (VDD), U18.27 (VDD), U18.41 (VDD), U18.5 (VDD), U18.51 (VDD), U18.58 (VDD), U18.92 (VDD)
- no-connect marks 52 -> 1
Other:
- note removed: "3.3V - 620mA"
- moved on the sheet: U1, U2

Commit message: added decoupling for DSP
Parts:
- added C112, C113, C114, C115, C149, C150, C151, C152: 2.2uF, PCM_JLCPCB:C_0402, symbol PCM_JLCPCB-Capacitors:0402,2.2uF
- added C116, C118, C127: 1uF, PCM_JLCPCB:C_0402, symbol PCM_JLCPCB-Capacitors:0402,1uF
- added C117, C119, C121, C122, C123, C124, C125, C126, C128, C129, C130, C131, C132, C133, C134, C136, C137, C138, C140, C141, C142, C143, C144, C145, C146: 100nF, PCM_JLCPCB:C_0402, symbol PCM_JLCPCB-Capacitors:0402,100nF
- added C120, C135, C139, C148: 4.7uF, PCM_JLCPCB:C_0402, symbol PCM_JLCPCB-Capacitors:0402,4.7uF
- added C147, C153: 10uF, PCM_JLCPCB:C_0603, symbol PCM_JLCPCB-Capacitors:0603,10uF
- added C154: 220pF, PCM_JLCPCB:C_0402, symbol PCM_JLCPCB-Capacitors:0402,220pF
- added L6: 2.2u, symbol Device:L
- added R116: 1kΩ, PCM_JLCPCB:R_0402, symbol PCM_JLCPCB-Resistors:0402,1kΩ
- added R117: 10kΩ, PCM_JLCPCB:R_0402, symbol PCM_JLCPCB-Resistors:0402,10kΩ
Connections:
- net +3.3V is gone; now on net VBAT: R15.1, R19.1, U1.1 (VDD), U1.14 (VDD), U1.27 (VDD), U1.3 (VDDQ), U1.43 (VDDQ), U1.49 (VDDQ), U1.9 (VDDQ), U2.8 (VCC), U3.8 (VDD), Y1.1 (Standby), Y1.4 (VDD)
- net VTREF is gone; now on net VBAT: U18.1 (VBAT), U18.116 (VDD), U18.12 (VDD), U18.128 (VDD), U18.141 (VDD), U18.157 (VDD), U18.169 (VDD), U18.27 (VDD), U18.41 (VDD), U18.5 (VDD), U18.51 (VDD), U18.58 (VDD), U18.92 (VDD)
- net FLASH_~{CS}: now also R117.2
- net FRAM_WP: now also R116.2
- net GND: now also U1.12 (VSSQ), U1.28 (VSS), U1.41 (VSS), U1.46 (VSSQ), U1.52 (VSSQ), U1.54 (VSS), U1.6 (VSSQ), U18.33 (VREFM), C112.2, C113.2, C114.2, C115.2, C116.2, C117.2, C118.2, C119.2, C120.2, C121.2, C122.2, C123.2, C124.2, C125.2, C126.2, C127.2, C128.2, C129.2, C130.2, C131.2, C132.2, C133.2, C134.2, C135.2, C136.2, C137.2, C138.2, C139.2, C140.2, C141.2, C142.2, C143.2, C144.2, C145.2, C146.2, C147.2, C148.2, C149.2, C150.2, C151.2, C152.2, C153.2, C154.2
- net GNDD: no longer U1.12 (VSSQ), U1.28 (VSS), U1.41 (VSS), U1.46 (VSSQ), U1.52 (VSSQ), U1.54 (VSS), U1.6 (VSSQ)
- net VBAT: now reaches U18.105 (VDDXSPI2)
- net VBAT: now also U18.110 (VDDXSPI2), U18.127 (VDDLDO), U18.146 (VDD50USB), U18.147 (VDD33USB), U18.15 (VDDSMPS), U18.168 (VDDLDO), U18.35 (VDDA), U18.59 (VDDLDO), U18.63 (VDDXSPI1), U18.69 (VDDXSPI1), U18.75 (VDDXSPI1), U18.81 (VDDXSPI1), U18.91 (VDDLDO), U18.93 (VDDXSPI2), U18.99 (VDDXSPI2), C116.1, C117.1, C118.1, C119.1, C120.1, C121.1, C122.1, C123.1, C124.1, C125.1, C126.1, C127.1, C128.1, C129.1, C130.1, C131.1, C132.1, C133.1, C134.1, C135.1, C136.1, C137.1, C138.1, C139.1, C140.1, C141.1, C142.1, C143.1, C144.1, C145.1, C146.1, C147.1, C148.1, R116.1, R117.1
- net at U18.125 (VCAP3): now also C113.1
- net VLXSMPS: now reaches U18.14 (VLXSMPS)
- net VLXSMPS: now also C154.1, L6.2
- net VFBSMPS: now reaches U18.16 (VFBSMPS)
- net VFBSMPS: now also C149.1, C150.1, C151.1, C152.1, C153.1, L6.1
- net at U18.166 (VCAP4): now also C112.1
- net at U18.61 (VCAP1): now also C115.1
- net at U18.89 (VCAP2): now also C114.1
Other:
- moved on the sheet: U3, Y1

Commit message: commit
Parts:
- added C155: 100nF, PCM_JLCPCB:C_0402, symbol PCM_JLCPCB-Capacitors:0402,100nF
- added R35, R40, R45: 33Ω, PCM_JLCPCB:R_0402, symbol PCM_JLCPCB-Resistors:0402,33Ω
Connections:
- net VFBSMPS is gone; now on net VCAP: C149.1, C150.1, C151.1, C152.1, C153.1, L6.1, U18.16 (VFBSMPS)
- net GND: now also C155.2
- net SWCLK: now also R40.2; no longer U18.123 (PA14(JTCK)
- net SWDIO: now also R35.2; no longer U18.122 (PA13(JTMS)
- net SWO: now also R45.2; no longer U18.163 (PB3(JTDO)
- net VBAT: now also C155.1; no longer C143.1, C144.1, C145.1, C146.1, U18.127 (VDDLDO), U18.168 (VDDLDO), U18.59 (VDDLDO), U18.91 (VDDLDO)
- net VCAP: now reaches C113.1, U18.125 (VCAP3)
- net VCAP: now also C112.1, C114.1, C115.1, C143.1, C144.1, C145.1, C146.1, U18.127 (VDDLDO), U18.166 (VCAP4), U18.168 (VDDLDO), U18.59 (VDDLDO), U18.61 (VCAP1), U18.89 (VCAP2), U18.91 (VDDLDO)
- net MIDI_UART0_TX: no longer names the net of U18.121 (PA12)
- new net: R35.1, U18.122 (PA13(JTMS)
- new net: R40.1, U18.123 (PA14(JTCK)
- new net: R45.1, U18.163 (PB3(JTDO)
Other:
- moved on the sheet: C149, C150, C151, C152, C153, C154, L6

Commit message: started the layout process
Parts:
- removed C129, C131: 100nF, PCM_JLCPCB:C_0402, symbol PCM_JLCPCB-Capacitors:0402,100nF
- added C67, C76, C77: 100nF, PCM_JLCPCB:C_0402, symbol PCM_JLCPCB-Capacitors:0402,100nF
- added NT1, NT10, NT3, NT4, NT5, NT6, NT7, NT8, NT9: ~, NetTie:NetTie-2_SMD_Pad0.5mm, symbol Device:NetTie_2
- U2: footprint Package_SO:SOIC-8_5.23x5.23mm_P1.27mm -> Package_SO:SOIC-8_5.3x5.3mm_P1.27mm
Connections:
- net GND: now also C67.2, C76.2, C77.2
- net VBAT: now also NT9.2; no longer C116.1, C117.1, C120.1, C121.1, C122.1, C123.1, C124.1, C125.1, C126.1, C127.1, C128.1, C130.1, C132.1, C133.1, C134.1, C135.1, C136.1, C137.1, C138.1, C139.1, C140.1, C141.1, C142.1, C147.1, C148.1, C155.1, R116.1, R117.1, R15.1, R19.1, U1.1 (VDD), U1.14 (VDD), U1.27 (VDD), U1.3 (VDDQ), U1.43 (VDDQ), U1.49 (VDDQ), U1.9 (VDDQ), U18.105 (VDDXSPI2), U18.110 (VDDXSPI2), U18.116 (VDD), U18.12 (VDD), U18.128 (VDD), U18.141 (VDD), U18.146 (VDD50USB), U18.147 (VDD33USB), U18.15 (VDDSMPS), U18.157 (VDD), U18.169 (VDD), U18.27 (VDD), U18.35 (VDDA), U18.41 (VDD), U18.5 (VDD), U18.51 (VDD), U18.58 (VDD), U18.63 (VDDXSPI1), U18.69 (VDDXSPI1), U18.75 (VDDXSPI1), U18.81 (VDDXSPI1), U18.92 (VDD), U18.93 (VDDXSPI2), U18.99 (VDDXSPI2), U2.8 (VCC), U3.8 (VDD), Y1.1 (Standby), Y1.4 (VDD)
- net VCAP: now also NT5.1; no longer C143.1, C144.1, C145.1, C146.1, U18.127 (VDDLDO), U18.168 (VDDLDO), U18.59 (VDDLDO), U18.91 (VDDLDO)
- new net +3.3V: C155.1, C67.1, NT1.1, NT10.1, NT3.1, NT4.1, NT6.1, NT7.1, NT8.1, NT9.1, R116.1, R117.1, R15.1, R19.1, U1.1 (VDD), U1.14 (VDD), U1.27 (VDD), U1.3 (VDDQ), U1.43 (VDDQ), U1.49 (VDDQ), U1.9 (VDDQ), U2.8 (VCC), U3.8 (VDD), Y1.1 (Standby), Y1.4 (VDD)
- new net VDD: C120.1, C121.1, C122.1, C123.1, C124.1, C125.1, C126.1, C128.1, C130.1, C132.1, C133.1, C76.1, C77.1, NT1.2, U18.116 (VDD), U18.12 (VDD), U18.128 (VDD), U18.141 (VDD), U18.157 (VDD), U18.169 (VDD), U18.27 (VDD), U18.41 (VDD), U18.5 (VDD), U18.51 (VDD), U18.58 (VDD), U18.92 (VDD)
- new net VDD33USB: C116.1, C117.1, NT10.2, U18.146 (VDD50USB), U18.147 (VDD33USB)
- new net VDDA: C127.1, C134.1, NT3.2, U18.35 (VDDA)
- new net VDDLDO: C143.1, C144.1, C145.1, C146.1, NT5.2, U18.127 (VDDLDO), U18.168 (VDDLDO), U18.59 (VDDLDO), U18.91 (VDDLDO)
- new net VDDSMPS: C147.1, C148.1, NT6.2, U18.15 (VDDSMPS)
- new net VDDXSPI1: C135.1, C136.1, C137.1, C138.1, NT4.2, U18.63 (VDDXSPI1), U18.69 (VDDXSPI1), U18.75 (VDDXSPI1), U18.81 (VDDXSPI1)
- new net VDDXSPI2: C139.1, C140.1, C141.1, C142.1, NT7.2, U18.105 (VDDXSPI2), U18.110 (VDDXSPI2), U18.93 (VDDXSPI2), U18.99 (VDDXSPI2)
- new net VTREF: NT8.2
Other:
- moved on the sheet: C116, C117, C118, C119, C139, C140, C141, C142, C147, C148

Commit message: lot of changes
Parts:
- added C14, C58, C64, C73: 1uF, PCM_JLCPCB:C_0402, symbol PCM_JLCPCB-Capacitors:0402,1uF
- added C59: 100nF, PCM_JLCPCB:C_0402, symbol PCM_JLCPCB-Capacitors:0402,100nF
- added D2: SMF6.0CA, PCM_JLCPCB:D_SOD-123FL, symbol PCM_JLCPCB-Diodes:TVS-Bi,SMF6.0CA
- added L1: Choke_Wurth_WE-CNSW_744232090, Inductor_SMD:L_CommonMode_Wurth_WE-CNSW-1206, symbol Filter:Choke_Wurth_WE-CNSW_744232090
- added R10, R11: 56kΩ, PCM_JLCPCB:R_0402, symbol PCM_JLCPCB-Resistors:0402,56kΩ
- added R2: 220Ω, PCM_JLCPCB:R_0805, symbol PCM_JLCPCB-Resistors:0805,220Ω
- added R36: 4.7kΩ, PCM_JLCPCB:R_0402, symbol PCM_JLCPCB-Resistors:0402,4.7kΩ
- added R39: 10kΩ, PCM_JLCPCB:R_0402, symbol PCM_JLCPCB-Resistors:0402,10kΩ
- added R5: 2kΩ, PCM_JLCPCB:R_0402, symbol PCM_JLCPCB-Resistors:0402,2kΩ
- added R98: 47Ω, PCM_JLCPCB:R_0402, symbol PCM_JLCPCB-Resistors:0402,47Ω
- added U12: USBLC6-2P6, Package_TO_SOT_SMD:SOT-666, symbol Power_Protection:USBLC6-2P6
- added U15: ISOM8115, Package_SO:SOIC-4_4.55x2.6mm_P1.27mm, symbol Isolator:EL814
Connections:
- net GNDD is gone; now on net GND: U2.4 (GND)
- net +3.3V: now also R5.1
- net D+: now also U12.6 (I/O1); no longer U18.149 (PM11)
- net D-: now also U12.4 (I/O2); no longer U18.148 (PM12)
- net GND: now also C14.2, C58.2, C64.2, C73.2, D2.1, R10.2, R11.2, R39.2, U12.2 (GND)
- net VDDA: no longer U18.35 (VDDA)
- net 2.5V_VREF: no longer names the net of U18.34 (VREFP)
- net 2.5V_VREF: now also C58.1, C59.1, R98.2
- net MIDI_UART0_RX renamed UART0_RX
- net UART0_RX: now also R5.2, U15.4
- net SPDIF_OUT renamed SPDIF_NOT_USED
- net VBUS_detect renamed VBUS_DETECT
- net VBUS_DETECT: now also C64.1, R36.2, R39.1
- new net: L1.2, U12.1 (I/O1)
- new net: L1.3, U12.3 (I/O2)
- new net: R2.2, U15.2
- new net +2.5VA: R98.1, U18.35 (VDDA)
- new net CC: R10.1
- new net D+_filt: L1.1, U18.149 (PM11)
- new net D-_filt: L1.4, U18.148 (PM12)
- new net GNDPWR: U15.3
- new net MIDI IN Shield: C73.1, D2.2
- new net Midi In Sink: R2.1
- new net Midi In Source: U15.1
- new net VBUS: C14.1, R36.1, U12.5 (VBUS)
- new net VCONN: R11.1
- no-connect marks 1 -> 2
Other:
- moved on the sheet: C67, R117, U2, U3

Commit message: last stm32h7 version
Parts:
- added J301: Conn_ARM_JTAG_SWD_20, Connector_PinSocket_1.27mm:PinSocket_2x10_P1.27mm_Horizontal, symbol Connector:Conn_ARM_JTAG_SWD_20
- added U301: STM32N657I0H3Q, User:VFBGA178_12X12_STM, symbol User:STM32N657I0H3Q
- L6: footprint (none) -> Inductor_SMD:L_1206_3216Metric
Connections:
- net GNDPWR is gone; now on net GND: U15.3
- new net: J301.10 (GND), J301.12 (GND), J301.14 (GND), J301.16 (GND), J301.18 (GND), J301.20 (GND), J301.4 (GND), J301.6 (GND), J301.8 (GND)
