File: MCU.kicad_sch (KiCad schematic)
At the start: 48 parts, among them IC2 R7KA8P1KFLCAB#UC0, J1 UI Board Connector, U1 W9825G6KH-6, U10 ISOUSB111DWXR, U12 USBLC6-2P6, U2 IS25LX512M-JHLE, U3 FM24CL64B, Y1 ASDLJ-E-24.576MHZ-L-R-T, Y3 SG-5032CAN 24MHz

Commit message: progressed with the layout
Other:
- note removed: "ADD load switch!!!"
- note removed: "TPS22919"
Changed lines of the file:
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@@
+	)
+	(rectangle
+		(start 231.14 182.88)
+		(end 293.37 231.14)
+		(stroke
+			(width 0)
+			(type dash)
+		)
+		(fill
+			(type none)
+		)
 	)
 	(rectangle
@@
 			(width 0)
 			(type dash)
-		)
-		(fill
-			(type none)
-		)
-	)
-	(rectangle
-		(start 236.22 184.15)
-		(end 298.45 233.68)
-		(stroke
-			(width 0.254)
-			(type solid)
-			(color 255 0 0 1)
 		)
 		(fill
@@
 		)
 	)
-	(text "ADD load switch!!!"
-		(exclude_from_sim no)
-		(at 248.158 193.294 0)
-		(effects
-			(font
-				(size 1.27 1.27)
-				(thickness 0.254)
-				(bold yes)
-				(color 255 0 0 1)
-			)
-		)
-	)
 	(text "Preset FRAM"
 		(exclude_from_sim no)
@@
 		(effects
 			(font
-				(size 2.54 2.54)
-			)
-		)
-	)
-	(text "TPS22919"
-		(exclude_from_sim no)
-		(at 262.382 212.598 0)
-		(effects
-			(font
