File: ProjectY.kicad_pcb (KiCad board)
At the start: 4 copper layers, 100 x 85 mm, 254 parts, among them J2 Conn_ARM_JTAG_SWD_10, J3 9V, J5 Out, J6 IN, J7 MIDI In, J9 USB_C_Receptacle_USB2.0_14P, U1 W9825G6KH-6, U10 RT8293B, U12 USBLC6-2P6, U14 TPS26400PWPR, U15 ISOM8115, U18 STM32H7R7I8Tx, U2 W25Q128JVS, U201 OPA1678, U202 OPA1678, U203 OPA1678, U204 OPA1678, U205 TAC5242, U206 OPA1678, U22 TLV77325PDBVR, U3 FM24CL64B, U4 TPS7A39, U5 TPS560430XFDBVT, Y1 ASDLJ-E-49.152MHZ-L-R-T

Commit message: last stm32h7 version
Parts:
- removed C106, C107, C53, C56: 100uF, PCM_JLCPCB:C_1206
- removed C26, C33, C41, C42, C48, C49, C5, C7: 10uF, PCM_JLCPCB:C_0603
- removed R119: 110k, Resistor_SMD:R_0402_1005Metric
- removed R120: 8.2k, Resistor_SMD:R_0402_1005Metric
- removed R130: 12k, Resistor_SMD:R_0402_1005Metric
- removed R131: 20k, Resistor_SMD:R_0402_1005Metric
- added C131: 47uF, PCM_JLCPCB:C_1206, F.Cu at (182.9, 116.7)
- added C156: 47uF, PCM_JLCPCB:C_1206, F.Cu at (182.9, 114.3)
- added C157: 47uF, PCM_JLCPCB:C_1206, F.Cu at (182.9, 112.0)
- added C158: 47uF, PCM_JLCPCB:C_1206, F.Cu at (182.9, 109.6)
- added C401: 1uF, PCM_JLCPCB:C_0402, F.Cu at (185.7, 100.9)
- added C402: 10uF, PCM_JLCPCB:C_0603, F.Cu at (187.6, 101.2)
- added C403: 10uF, PCM_JLCPCB:C_0603, F.Cu at (183.8, 99.9)
- added C404: 10uF, PCM_JLCPCB:C_0603, F.Cu at (187.6, 99.9)
- added C405: 10uF, PCM_JLCPCB:C_0603, F.Cu at (183.8, 101.2)
- added J15: 009155002852006, User:KYO_009155002852006, B.Cu at (237.6, 96.6)
- added J16: 009155002852006, User:KYO_009155002852006, B.Cu at (230.1, 96.6)
- added J301: Conn_ARM_JTAG_SWD_20, Connector_PinSocket_1.27mm:PinSocket_2x10_P1.27mm_Horizontal, F.Cu at (188.5, 176.9)
- added L6: 2.2u, Inductor_SMD:L_1206_3216Metric, F.Cu at (2.38, 1.23)
- added R401: 110kΩ, PCM_JLCPCB:R_0603, F.Cu at (238.6, 109.4)
- added R402: 8.2kΩ, PCM_JLCPCB:R_0402, F.Cu at (236.3, 109.6)
- added R403: 12kΩ, PCM_JLCPCB:R_0402, F.Cu at (234.4, 109.6)
- added R404: 20kΩ, PCM_JLCPCB:R_0402, F.Cu at (235.8, 118.6)
- added U301: STM32N657I0H3Q, User:VFBGA178_12X12_STM, F.Cu at (94.9, 147.2)
- C108, C109, C110, C111: value 100uF -> 47uF
- R217, R218, R219, R220: footprint PCM_JLCPCB:R_0805 -> PCM_JLCPCB:R_0402
- U5: value TPS560430XFDBVT -> TI LMR54406DBVR
- moved C118 161.8 mm to (179.6, 133.2), turned to 90 degrees
- moved C119 160.5 mm to (180.6, 133.2), turned to 90 degrees
- moved C126 159.5 mm to (180.1, 135.6), turned to 180 degrees
- moved C125 157.3 mm to (180.2, 139.2), turned to 180 degrees
- moved C155 157.0 mm to (179.3, 141.7), turned to 180 degrees
- moved C154 156.7 mm to (180.2, 140.2), turned to 180 degrees
- moved C3 156.1 mm to (241.1, 110.8), turned to 90 degrees
- moved Y1 155.8 mm to (179.3, 143.9), turned to -90 degrees
- moved U204 155.5 mm to (172.4, 123.3), turned to 180 degrees
- moved C120 154.6 mm to (187.4, 129.7), turned to 90 degrees
- moved C145 153.5 mm to (188.3, 129.7), turned to 90 degrees
- moved C124 153.2 mm to (180.1, 146.7), turned to 180 degrees
- moved C115 152.3 mm to (189.2, 129.7), turned to 90 degrees
- moved C4 151.7 mm to (235.8, 119.5), turned to 180 degrees
- moved C123 149.9 mm to (180.1, 153.7), turned to 180 degrees
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Connections:
- C109 pad 1: GND -> /Analog Audio/+V_OPA
- C109 pad 2: /Analog Audio/-V_OPA -> GND
- C111 pad 1: GND -> /Analog Audio/+V_OPA
- C111 pad 2: /Analog Audio/-V_OPA -> GND
- C129 pad 1: Net-(C129-Pad1) -> +9VA
- C205 pad 1: Net-(C203-Pad2) -> ADC_R-
- C205 pad 2: ADC_L- -> Net-(C203-Pad2)
- C206 pad 1: Net-(C203-Pad1) -> ADC_R+
- C206 pad 2: ADC_L+ -> Net-(C203-Pad1)
- C207 pad 1: Net-(C204-Pad2) -> ADC_L-
- C207 pad 2: ADC_R- -> Net-(C204-Pad2)
- C208 pad 1: Net-(C204-Pad1) -> ADC_L+
- C208 pad 2: ADC_R+ -> Net-(C204-Pad1)
- D3 pad 2: Net-(C129-Pad1) -> +9VA
- J7 pad RN: unconnected-(J7-PadRN) -> /DSP/MIDI IN Shield
- J7 pad SN: unconnected-(J7-PadSN) -> /DSP/MIDI IN Shield
- J7 pad TN: unconnected-(J7-PadTN) -> /DSP/MIDI IN Shield
- R205 pad 1: Net-(U201B--) -> Net-(U201A--)
- R206 pad 1: Net-(U201B--) -> Net-(U201A--)
- R208 pad 1: Net-(U201A--) -> Net-(U201B--)
- R209 pad 1: Net-(U201A--) -> Net-(U201B--)
- U14 pad 15: Net-(C129-Pad1) -> +9VA
- U14 pad 16: Net-(C129-Pad1) -> +9VA
- U15 pad 3: GNDPWR -> GND
- U4 pad 1: Net-(U4-INP) -> +9VA
- U4 pad 2: unconnected-(U4-EN-Pad2) -> +9VA
- U4 pad 3: unconnected-(U4-NR/SS-Pad3) -> Net-(U4-NR/SS)
Routing:
- net Net-(U203B--): track 0.00 -> 0.65 mm
- net Net-(U203A--): track 0.00 -> 0.65 mm

Commit message: imrt1176 is added
Parts:
- removed C112, C113, C114, C115, C149, C150, C151, C152: 2.2uF, PCM_JLCPCB:C_0402
- removed C116, C118, C127, C58, C64, C73: 1uF, PCM_JLCPCB:C_0402
- removed C117, C119, C121, C122, C123, C124, C125, C126, C128, C130, C132, C133, C134, C136, C137, C138, C140, C141, C142, C143, C144, C145, C146, C155, C76, C77: 100nF, PCM_JLCPCB:C_0402
- removed C120, C135, C139, C148: 4.7uF, PCM_JLCPCB:C_0402
- removed C129, C147, C153: 10uF, PCM_JLCPCB:C_0603
- removed C154: 220pF, PCM_JLCPCB:C_0402
- removed C63, C68, C69, C80, C85: 10uF, PCM_JLCPCB:C_0402
- removed D2: SMF6.0CA, PCM_JLCPCB:D_SOD-123FL
- removed D3: SMF20CA, PCM_JLCPCB:D_SOD-123FL
- removed J301: Conn_ARM_JTAG_SWD_20, Connector_PinSocket_1.27mm:PinSocket_2x10_P1.27mm_Horizontal
- removed L6: 2.2u, Inductor_SMD:L_1206_3216Metric
- removed NT1, NT10, NT3, NT4, NT5, NT6, NT7, NT8, NT9: ~, NetTie:NetTie-2_SMD_Pad0.5mm
- removed R116: 1kΩ, PCM_JLCPCB:R_0402
- removed R32: 100kΩ, PCM_JLCPCB:R_0402
- removed R33: 22kΩ, PCM_JLCPCB:R_0402
- removed R34, R98: 47Ω, PCM_JLCPCB:R_0402
- removed R35, R40, R45: 33Ω, PCM_JLCPCB:R_0402
- removed R36: 4.7kΩ, PCM_JLCPCB:R_0402
- removed R39: 10kΩ, PCM_JLCPCB:R_0402
- removed R401: 110kΩ, PCM_JLCPCB:R_0603
- removed R402: 8.2kΩ, PCM_JLCPCB:R_0402
- removed R403: 12kΩ, PCM_JLCPCB:R_0402
- removed R404: 20kΩ, PCM_JLCPCB:R_0402
- removed R46: 75kΩ, PCM_JLCPCB:R_0402
- removed R47: 24kΩ, PCM_JLCPCB:R_0402
- removed U10: RT8293B, Package_SO:TI_SO-PowerPAD-8
- removed U15: ISOM8115, Package_SO:SOIC-4_4.55x2.6mm_P1.27mm
- removed U18: STM32H7R7I8Tx, Package_QFP:LQFP-176_24x24mm_P0.5mm
- removed U22: TLV77325PDBVR, Package_TO_SOT_SMD:SOT-23-5
- removed U301: STM32N657I0H3Q, User:VFBGA178_12X12_STM
- added C1: 10uF, PCM_JLCPCB:C_0402, F.Cu at (238.9, 122.2)
- added C11: 220nF, PCM_JLCPCB:C_0402, F.Cu at (176.8, 33.0)
- added C12: 47uF, PCM_JLCPCB:C_1206, F.Cu at (139.8, 47.3)
- added C13: 47uF, PCM_JLCPCB:C_1206, F.Cu at (139.8, 49.2)
- added C15: 1uF, PCM_JLCPCB:C_0402, F.Cu at (213.0, 32.2)
- added C16: 1uF, PCM_JLCPCB:C_0402, F.Cu at (213.0, 34.0)
- added C17: 2.2nF, PCM_JLCPCB:C_0805, F.Cu at (198.7, 37.1)
- added C18: 2.2nF, PCM_JLCPCB:C_0805, F.Cu at (198.7, 40.1)
- added C19: 10uF, PCM_JLCPCB:C_0402, F.Cu at (195.1, 30.4)
- added C2: 10uF, PCM_JLCPCB:C_0402, F.Cu at (238.9, 124.0)
- added C20: 10uF, PCM_JLCPCB:C_0402, F.Cu at (195.1, 32.2)
- added C21: 10uF, PCM_JLCPCB:C_0402, F.Cu at (195.1, 34.0)
- added C22: 10uF, PCM_JLCPCB:C_0402, F.Cu at (195.1, 35.9)
- added C23: 10uF, PCM_JLCPCB:C_0402, F.Cu at (195.1, 37.8)
- added C241: 10uF, PCM_JLCPCB:C_0402, F.Cu at (139.8, 64.1)
- added C26: 10u, Capacitor_SMD:C_1206_3216Metric, F.Cu at (181.2, 52.1)
- added C31: 220n, Capacitor_SMD:C_0603_1608Metric, F.Cu at (162.6, 43.4)
- added C32: 22u, Capacitor_SMD:C_0805_2012Metric, F.Cu at (183.3, 33.6)
- added C33: 22u, Capacitor_SMD:C_0805_2012Metric, F.Cu at (183.3, 36.6)
- added C34: 4n7, Capacitor_SMD:C_0603_1608Metric, F.Cu at (166.6, 33.3)
- added C36: 10uF, PCM_JLCPCB:C_0402, F.Cu at (193.1, 67.5)
- added C37: 10uF, PCM_JLCPCB:C_0402, F.Cu at (193.1, 69.4)
- added C38: 10uF, PCM_JLCPCB:C_0402, F.Cu at (195.9, 60.1)
- added C39: 10uF, PCM_JLCPCB:C_0402, F.Cu at (195.9, 62.0)
- added C40: 2.2uF, PCM_JLCPCB:C_0402, F.Cu at (195.9, 63.8)
- added C41: 4.7uF, PCM_JLCPCB:C_0402, F.Cu at (195.9, 65.7)
- added C42: 2.2uF, PCM_JLCPCB:C_0402, F.Cu at (195.9, 67.5)
- added C43: 2.2uF, PCM_JLCPCB:C_0402, F.Cu at (195.9, 69.4)
- added C44: 10uF, PCM_JLCPCB:C_0402, F.Cu at (198.8, 60.1)
- added C45: 2.2uF, PCM_JLCPCB:C_0402, F.Cu at (198.8, 62.0)
- added C46: 100nF, PCM_JLCPCB:C_0402, F.Cu at (175.4, 59.2)
- added C47: 2.2uF, PCM_JLCPCB:C_0402, F.Cu at (198.8, 63.8)
- added C48: 10uF, PCM_JLCPCB:C_0402, F.Cu at (195.1, 39.6)
- added C49: 10uF, PCM_JLCPCB:C_0402, F.Cu at (195.1, 41.5)
- added C5: 10uF, PCM_JLCPCB:C_0402, F.Cu at (238.9, 125.9)
- added C53: 100nF, PCM_JLCPCB:C_0603, F.Cu at (202.9, 41.3)
- added C56: 100nF, PCM_JLCPCB:C_0603, F.Cu at (202.9, 43.6)
- added C62: 10uF, PCM_JLCPCB:C_0402, F.Cu at (176.8, 34.8)
- added C7: 10uF, PCM_JLCPCB:C_0402, F.Cu at (174.0, 36.7)
- added C8: 100nF, PCM_JLCPCB:C_0402, F.Cu at (174.0, 38.5)
- added D4: B5819W, Diode_SMD:D_SOD-123, F.Cu at (175.5, 48.7)
- added D5: B5819W, Diode_SMD:D_SOD-123, F.Cu at (175.5, 52.1)
- added J17: Out, User:Jack_6.35mm_Neutrik_NRJ6HF_Horizontal, F.Cu at (196.4, 113.2)
- added L3: 3.5u, Inductor_SMD:L_12x12mm_H8mm, F.Cu at (244.8, 51.7)
- added Q2: AO3401A, Package_TO_SOT_SMD:SOT-23, F.Cu at (168.2, 54.1)
- added R13: 1kΩ, PCM_JLCPCB:R_0402, F.Cu at (175.4, 64.8)
- added R14: 1kΩ, PCM_JLCPCB:R_0402, F.Cu at (175.4, 66.6)
- added R16: 1kΩ, PCM_JLCPCB:R_0402, F.Cu at (175.4, 68.5)
- added R17: 33kΩ, PCM_JLCPCB:R_0402, F.Cu at (176.8, 40.4)
- added R18: 100kΩ, PCM_JLCPCB:R_0402, F.Cu at (148.3, 47.3)
- added R20: 10kΩ, PCM_JLCPCB:R_0402, F.Cu at (148.3, 51.0)
- added R21: 10kΩ, PCM_JLCPCB:R_0402, F.Cu at (148.3, 52.9)
- added R22: 1MΩ, PCM_JLCPCB:R_0402, F.Cu at (123.1, 107.1)
- added R23: 100, Resistor_SMD:R_0603_1608Metric, F.Cu at (166.6, 35.8)
- added R24: 1M, Resistor_SMD:R_0603_1608Metric, F.Cu at (166.6, 38.3)
- added R25: 110k, Resistor_SMD:R_0603_1608Metric, F.Cu at (166.6, 40.8)
- added R26: 100k, Resistor_SMD:R_0603_1608Metric, F.Cu at (166.6, 43.4)
- added R27: 1M, Resistor_SMD:R_0603_1608Metric, F.Cu at (170.6, 33.3)
- added R28: 12k, Resistor_SMD:R_0603_1608Metric, F.Cu at (170.6, 35.8)
- added R29: 12k, Resistor_SMD:R_0603_1608Metric, F.Cu at (170.6, 38.3)
- added R7: 4.7kΩ, PCM_JLCPCB:R_0402, F.Cu at (176.8, 36.7)
- added R8: 24kΩ, PCM_JLCPCB:R_0402, F.Cu at (145.4, 51.0)
- added R9: 4.7kΩ, PCM_JLCPCB:R_0402, F.Cu at (175.4, 62.9)
- added U11: RT8293B, Package_SO:SOP-8-1EP_4.57x4.57mm_P1.27mm_EP4.57x4.45mm_ThermalVias, F.Cu at (207.3, 25.1)
- added U13: LM74700, Package_TO_SOT_SMD:SOT-23-6, F.Cu at (203.5, 38.0)
- added U6: MIMXRT1176CVM8A, User:BGA289C80P17X17_1400X1400X152, F.Cu at (209.1, 155.2)
- added U8: TLV77325PDBVR, Package_TO_SOT_SMD:SOT-23-5, F.Cu at (163.1, 54.1)
- added U9: TL431DBZ, Package_TO_SOT_SMD:SOT-23, F.Cu at (212.1, 75.8)
- added Y3: SG-5032CAN 24MHz, Oscillator:Oscillator_SMD_SeikoEpson_SG8002LB-4Pin_5.0x3.2mm, F.Cu at (180.3, 60.9)
- C10, C6, C9: value 100nF -> 10uF
- C24: value 4.7uF -> 10uF; footprint PCM_JLCPCB:C_0805 -> PCM_JLCPCB:C_0402
- C25: value 1uF -> 10u; footprint PCM_JLCPCB:C_0402 -> Capacitor_SMD:C_1206_3216Metric
- C27: value 2.2nF -> 100n; footprint PCM_JLCPCB:C_0805 -> Capacitor_SMD:C_0603_1608Metric
- C28: value 100nF -> 10n; footprint PCM_JLCPCB:C_0402 -> Capacitor_SMD:C_0603_1608Metric
- C29: value DNP -> 6p8; footprint Capacitor_SMD:C_0805_2012Metric -> Capacitor_SMD:C_0603_1608Metric
- C30: value C -> 8p2; footprint Capacitor_SMD:C_0402_1005Metric -> Capacitor_SMD:C_0603_1608Metric
- C4: value 1uF -> 100nF
- C57: value 10uF -> 100nF
- C59: value 100nF -> 1uF
- J2: footprint Connector_PinHeader_1.27mm:PinHeader_2x05_P1.27mm_Vertical_SMD -> Connector_PinHeader_2.54mm:PinHeader_1x02_P2.54mm_Vertical
- J5: value Out -> IN_R
- J6: value IN -> IN_L
- J7: value MIDI In -> Out
- L1: value Choke_Wurth_WE-CNSW_744232090 -> 4.7uH; footprint Inductor_SMD:L_CommonMode_Wurth_WE-CNSW-1206 -> Inductor_SMD:L_1206_3216Metric
- L4: value 3.6uH -> L; footprint Inductor_SMD:L_Cenker_CKCS8040 -> Inductor_SMD:L_CommonMode_Wurth_WE-CNSW-1206
- R1: value 0Ω -> 5.1kΩ
- R10: value 56kΩ -> 10kΩ
- R11: value 56kΩ -> 22kΩ; footprint PCM_JLCPCB:R_0402 -> PCM_JLCPCB:R_0805
- R15: value 1kΩ -> 5.1kΩ
- R19: value 1kΩ -> 10kΩ
- R2: value 220Ω -> 47Ω; footprint PCM_JLCPCB:R_0805 -> PCM_JLCPCB:R_0402
- R3: value 47Ω -> 10kΩ
- R31: value 24kΩ -> 1MΩ
- R5: value 2kΩ -> 75kΩ
- R6: value 4.3kΩ -> 10kΩ; footprint PCM_JLCPCB:R_0603 -> PCM_JLCPCB:R_0402
- U14: value TPS26400PWPR -> OPA1678; footprint User:PWP0016H-IPC_A -> Package_SO:SOIC-8_3.9x4.9mm_P1.27mm
- U5: value TI LMR54406DBVR -> TL431DBZ; footprint Package_TO_SOT_SMD:SOT-23-6 -> Package_TO_SOT_SMD:SOT-23
- Y1: value ASDLJ-E-49.152MHZ-L-R-T -> ASDLJ-E-24.576MHZ-L-R-T
- moved C14 165.9 mm to (213.0, 30.4)
- moved U5 151.4 mm to (212.1, 71.2)
- moved R3 129.9 mm to (209.1, 70.1)
- moved R6 126.9 mm to (209.1, 72.2)
- moved C10 126.4 mm to (174.0, 40.4)
- moved R12 123.9 mm to (176.8, 38.5)
- moved J2 121.8 mm to (204.9, 175.5), turned to -90 degrees
- moved C102 113.2 mm to (164.8, 61.1)
- moved C101 113.2 mm to (164.8, 59.2)
- moved C103 113.2 mm to (164.8, 62.9)
- moved C6 113.1 mm to (193.1, 60.1)
- moved C9 113.1 mm to (193.1, 62.0)
- moved R41 111.9 mm to (167.7, 61.1)
- moved U14 111.8 mm to (125.9, 102.9), turned to 0 degrees
- moved R19 111.3 mm to (148.3, 49.2)
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Connections:
- net FLASH_~{CS} renamed /DSP/FLASH_~{CS}
- C10 pad 1: GND -> +3.3V
- C10 pad 2: /DSP/~{RESET} -> GND
- C108 pad 1: /Analog Audio/+V_OPA -> +6.5V
- C109 pad 1: /Analog Audio/+V_OPA -> +6.5V
- C110 pad 1: /Analog Audio/+V_OPA -> +6.5V
- C111 pad 1: /Analog Audio/+V_OPA -> +6.5V
- C131 pad 2: /Analog Audio/-V_OPA -> -6.5V
- C14 pad 1: /DSP/VBUS -> Net-(U10-3.3V1)
- C14 pad 2: GND -> ISO_GND
- C156 pad 2: /Analog Audio/-V_OPA -> -6.5V
- C157 pad 2: /Analog Audio/-V_OPA -> -6.5V
- C158 pad 2: /Analog Audio/-V_OPA -> -6.5V
- C209 pad 1: /Analog Audio/+V_OPA -> +6.5V
- C210 pad 2: /Analog Audio/-V_OPA -> -6.5V
- C211 pad 1: /Analog Audio/+V_OPA -> +6.5V
- C212 pad 2: /Analog Audio/-V_OPA -> -6.5V
- C213 pad 1: /Analog Audio/+V_OPA -> +6.5V
- C214 pad 2: /Analog Audio/-V_OPA -> -6.5V
- C215 pad 1: /Analog Audio/+V_OPA -> +6.5V
- C216 pad 2: /Analog Audio/-V_OPA -> -6.5V
- C217 pad 1: /Analog Audio/+V_OPA -> +6.5V
- C218 pad 2: /Analog Audio/-V_OPA -> -6.5V
- C229 pad 1: /Analog Audio/+3.3V -> +3.3V
- C234 pad 1: Net-(U206B-+) -> Net-(U14B-+)
- C234 pad 2: Net-(U206B--) -> Net-(U14B--)
- C237 pad 1: Net-(U206B-+) -> Net-(U14B-+)
- C237 pad 2: Net-(U206B--) -> Net-(U14B--)
- C238 pad 1: Net-(U206A-+) -> Net-(U14A-+)
- C238 pad 2: Net-(U206A--) -> Net-(U14A--)
- C24 pad 1: GND -> 1.15V_DCDC
- C24 pad 2: -7V -> GND
- C240 pad 1: Net-(U206A-+) -> Net-(U14A-+)
- C240 pad 2: Net-(U206A--) -> Net-(U14A--)
- C25 pad 1: Net-(U10-SS/PG) -> +5V
- C28 pad 2: Net-(U10-SW) -> GND
- C29 pad 1: Net-(U10-COMP) -> +12V
- C29 pad 2: GND -> Net-(IC1-FBP)
- C3 pad 1: /PSU/+9V -> Net-(U11-BOOT)
- C3 pad 2: GND -> Net-(U11-SW)
- C30 pad 2: Net-(U10-FB) -> -12V
- C35 pad 1: /Analog Audio/+3.3V -> 1.15V_DCDC
- C4 pad 1: Net-(U14-dVdT) -> Net-(U11-SS/PG)
- C4 pad 2: PowerPad -> GND
- C57 pad 1: /Analog Audio/+3.3V -> GND
- C57 pad 2: GND -> /DSP/~{RESET}
- C59 pad 1: Net-(U18-VREFP) -> /DSP/VBUS
- C59 pad 2: unconnected-(C59-Pad2) -> ISO_GND
- C6 pad 1: Net-(U5-EN) -> 1.8V_DCDC
- C6 pad 2: -7V -> GND
- C66 pad 2: /Analog Audio/-V_OPA -> -6.5V
- C67 pad 1: /Analog Audio/+3.3V -> +3.3V
- C79 pad 1: /Analog Audio/+V_OPA -> +6.5V
- C9 pad 1: Net-(U5-CB) -> 1.8V_DCDC
- C9 pad 2: Net-(U5-SW) -> GND
- C99 pad 1: /Analog Audio/+3.3V -> +3.3V
- D1 pad 1: /PSU/+9V -> +9VA
- D201 pad 1: /Analog Audio/-V_OPA -> -5V_Clamp
- D201 pad 2: /Analog Audio/+V_OPA -> +5V_Clamp
- D202 pad 1: /Analog Audio/-V_OPA -> -5V_Clamp
- D202 pad 2: /Analog Audio/+V_OPA -> +5V_Clamp
- D203 pad 1: /Analog Audio/-V_OPA -> -5V_Clamp
- D203 pad 2: /Analog Audio/+V_OPA -> +5V_Clamp
- D204 pad 1: /Analog Audio/-V_OPA -> -5V_Clamp
- D204 pad 2: /Analog Audio/+V_OPA -> +5V_Clamp
- J2 pad 2: /DSP/SWDIO -> /DSP/JTAG_TMS
- J3 pad 2: /PSU/+9V -> +9VA
- J5 pad R: /Analog Audio/Line_Output_R -> GND
- J5 pad RN: unconnected-(J5-PadRN) -> GND
- J5 pad SN: unconnected-(J5-PadSN) -> GND
- J5 pad T: /Analog Audio/Line_Output_L -> /Analog Audio/IN_R
- J5 pad TN: unconnected-(J5-PadTN) -> /Analog Audio/IN_L
- J6 pad R: /Analog Audio/IN_R -> GND
- J7 pad R: /DSP/Midi In Source -> unconnected-(J7-PadR)
- J7 pad RN: /DSP/MIDI IN Shield -> unconnected-(J7-PadRN)
- J7 pad S: /DSP/MIDI IN Shield -> GND
- J7 pad SN: /DSP/MIDI IN Shield -> unconnected-(J7-PadSN)
- J7 pad T: /DSP/Midi In Sink -> /Analog Audio/Line_Output_L
- J7 pad TN: /DSP/MIDI IN Shield -> unconnected-(J7-PadTN)
- J9 pad A1: GND -> ISO_GND
- J9 pad A12: GND -> ISO_GND
- J9 pad B1: GND -> ISO_GND
- J9 pad B12: GND -> ISO_GND
- J9 pad S1: GND -> ISO_GND
- L1 pad 1: D+_filt -> Net-(L1-Pad1)
- L4 pad 1: Net-(U10-SW) -> Net-(Q1-D)
- L4 pad 2: /Analog Audio/+3.3V -> Net-(U11-VIN)
- R1 pad 1: GND -> /DSP/VCONN
- R1 pad 2: Net-(U18-BOOT0) -> ISO_GND
- R10 pad 1: /DSP/CC -> GND
- R10 pad 2: GND -> Net-(U9-REF)
- R11 pad 1: /DSP/VCONN -> Net-(C17-Pad2)
- R117 pad 1: /Analog Audio/+3.3V -> +3.3V
- R12 pad 1: +9-18V -> Net-(U11-VIN)
- R15 pad 1: /Analog Audio/+3.3V -> /DSP/CC
- R15 pad 2: FRAM_SDA -> ISO_GND
- R19 pad 1: /Analog Audio/+3.3V -> Net-(U9-REF)
- R19 pad 2: FRAM_SCL -> -5V_Clamp
- R2 pad 1: /DSP/Midi In Sink -> Net-(R2-Pad1)
- R203 pad 2: GND -> Net-(R203-Pad2)
- R204 pad 2: GND -> Net-(R204-Pad2)
- R221 pad 2: Net-(U206B--) -> Net-(U14B--)
- R222 pad 2: Net-(U206B-+) -> Net-(U14B-+)
- R223 pad 2: Net-(U206B-+) -> Net-(U14B-+)
- R224 pad 2: Net-(U206A--) -> Net-(U14A--)
- R225 pad 2: Net-(U206A-+) -> Net-(U14A-+)
- R226 pad 2: Net-(U206A-+) -> Net-(U14A-+)
- R227 pad 1: Net-(U206B--) -> Net-(U14B--)
- R228 pad 1: Net-(U206A--) -> Net-(U14A--)
- R229 pad 2: /Analog Audio/Line_Output_R -> unconnected-(R229-Pad2)
- R230 pad 2: /Analog Audio/Line_Output_L -> unconnected-(R230-Pad2)
- R3 pad 1: Net-(R3-Pad1) -> +5V_Clamp
- R3 pad 2: GND -> Net-(U5-REF)
- R31 pad 1: Net-(U5-FB) -> Net-(R203-Pad2)
- R31 pad 2: Net-(R3-Pad1) -> GND
- R5 pad 1: /Analog Audio/+3.3V -> Net-(R2-Pad1)
- R5 pad 2: UART0_RX -> Net-(U11-FB)
- R59 pad 1: /Analog Audio/+V_OPA -> +6.5V
- R6 pad 1: Net-(U5-FB) -> Net-(U5-REF)
- R6 pad 2: -7V -> GND
- R61 pad 2: /Analog Audio/-V_OPA -> -6.5V
- R74 pad 1: /Analog Audio/+3.3V -> +3.3V
- R84 pad 1: /Analog Audio/+3.3V -> +3.3V
- R86 pad 1: /Analog Audio/+3.3V -> +3.3V
- R92 pad 1: /Analog Audio/+3.3V -> +3.3V
- R94 pad 1: /Analog Audio/+3.3V -> +3.3V
- R95 pad 1: /Analog Audio/+3.3V -> +3.3V
- U1 pad 1: /Analog Audio/+3.3V -> +3.3V
- U1 pad 10: RAM_D5 -> /DSP/RAM_D5
- U1 pad 11: RAM_D6 -> /DSP/RAM_D6
- U1 pad 13: RAM_D7 -> /DSP/RAM_D7
- U1 pad 14: /Analog Audio/+3.3V -> +3.3V
- U1 pad 15: RAM_DQML -> /DSP/RAM_DQML
- U1 pad 16: RAM_~{WE} -> /DSP/RAM_~{WE}
- U1 pad 17: RAM_~{CAS} -> /DSP/RAM_~{CAS}
- U1 pad 18: RAM_~{RAS} -> /DSP/RAM_~{RAS}
- U1 pad 19: RAM_~{CS} -> /DSP/RAM_~{CS}
- U1 pad 2: RAM_D0 -> /DSP/RAM_D0
- U1 pad 20: RAM_BA0 -> /DSP/RAM_BA0
- U1 pad 21: RAM_BA1 -> /DSP/RAM_BA1
- U1 pad 22: RAM_A10 -> /DSP/RAM_A10
- U1 pad 23: RAM_A0 -> /DSP/RAM_A0
- U1 pad 24: RAM_A1 -> /DSP/RAM_A1
- U1 pad 25: RAM_A2 -> /DSP/RAM_A2
- U1 pad 26: RAM_A3 -> /DSP/RAM_A3
- U1 pad 27: /Analog Audio/+3.3V -> +3.3V
- U1 pad 29: RAM_A4 -> /DSP/RAM_A4
- U1 pad 3: /Analog Audio/+3.3V -> +3.3V
- U1 pad 30: RAM_A5 -> /DSP/RAM_A5
- U1 pad 31: RAM_A6 -> /DSP/RAM_A6
- U1 pad 32: RAM_A7 -> /DSP/RAM_A7
- U1 pad 33: RAM_A8 -> /DSP/RAM_A8
- U1 pad 34: RAM_A9 -> /DSP/RAM_A9
- U1 pad 35: RAM_A11 -> /DSP/RAM_A11
- U1 pad 36: RAM_A12 -> /DSP/RAM_A12
- U1 pad 37: RAM_CKE -> /DSP/RAM_CKE
- U1 pad 38: RAM_CLK -> /DSP/RAM_CLK
- U1 pad 39: RAM_DQMH -> /DSP/RAM_DQMH
- U1 pad 4: RAM_D1 -> /DSP/RAM_D1
- U1 pad 42: RAM_D8 -> /DSP/RAM_D8
- U1 pad 43: /Analog Audio/+3.3V -> +3.3V
- U1 pad 44: RAM_D9 -> /DSP/RAM_D9
- U1 pad 45: RAM_D10 -> /DSP/RAM_D10
- U1 pad 47: RAM_D11 -> /DSP/RAM_D11
- U1 pad 48: RAM_D12 -> /DSP/RAM_D12
- U1 pad 49: /Analog Audio/+3.3V -> +3.3V
- U1 pad 5: RAM_D2 -> /DSP/RAM_D2
- U1 pad 50: RAM_D13 -> /DSP/RAM_D13
- U1 pad 51: RAM_D14 -> /DSP/RAM_D14
- U1 pad 53: RAM_D15 -> /DSP/RAM_D15
- U1 pad 7: RAM_D3 -> /DSP/RAM_D3
- U1 pad 8: RAM_D4 -> /DSP/RAM_D4
- U1 pad 9: /Analog Audio/+3.3V -> +3.3V
- U12 pad 1: Net-(L1-Pad2) -> Net-(U10-UD-)
- U12 pad 2: GND -> ISO_GND
- U12 pad 3: Net-(L1-Pad3) -> Net-(U10-UD+)
- U12 pad 4: /DSP/D- -> /DSP/D+
- U12 pad 6: /DSP/D+ -> /DSP/D-
- U14 pad 1: /PSU/+9V -> Net-(R228-Pad2)
- U14 pad 2: /PSU/+9V -> Net-(U14A--)
- U14 pad 3: Net-(U14-UVLO) -> Net-(U14A-+)
- U14 pad 4: unconnected-(U14-NC-Pad4) -> -6.5V
- U14 pad 5: Net-(U14-OVP) -> Net-(U14B-+)
- U14 pad 6: unconnected-(U14-MODE-Pad6) -> Net-(U14B--)
- U14 pad 7: unconnected-(U14-SHDN_N-Pad7) -> Net-(R227-Pad2)
- U14 pad 8: PowerPad -> +6.5V
- U2 pad 2: FLASH_QSPI1 -> /DSP/FLASH_QSPI1
- U2 pad 3: FLASH_QSPI2 -> /DSP/FLASH_QSPI2
- U2 pad 5: FLASH_QSPI0 -> /DSP/FLASH_QSPI0
- U2 pad 6: FLASH_CLK -> /DSP/FLASH_CLK
- U2 pad 7: FLASH_QSPI3 -> /DSP/FLASH_QSPI3
- U2 pad 8: /Analog Audio/+3.3V -> +3.3V
- U201 pad 4: /Analog Audio/-V_OPA -> -6.5V
- U201 pad 8: /Analog Audio/+V_OPA -> +6.5V
- U202 pad 4: /Analog Audio/-V_OPA -> -6.5V
- U202 pad 8: /Analog Audio/+V_OPA -> +6.5V
- U203 pad 4: /Analog Audio/-V_OPA -> -6.5V
- U203 pad 8: /Analog Audio/+V_OPA -> +6.5V
- U204 pad 4: /Analog Audio/-V_OPA -> -6.5V
- U204 pad 8: /Analog Audio/+V_OPA -> +6.5V
- U205 pad 23: /Analog Audio/+3.3V -> Net-(U205-AVDD)
- U205 pad 4: /Analog Audio/I2S_SDI -> /Analog Audio/I2S_RX
- U205 pad 5: /Analog Audio/I2S_SDO -> /Analog Audio/I2S_TX
- U205 pad 6: /Analog Audio/+3.3V -> +3.3V
- U205 pad 7: /Analog Audio/+3.3V -> Net-(U205-AVDD)
- U205 pad 8: /Analog Audio/+3.3V -> Net-(U205-AVDD)
- U206 pad 1: Net-(R228-Pad2) -> unconnected-(U206-Pad1)
- U206 pad 2: Net-(U206A--) -> unconnected-(U206A---Pad2)
- U206 pad 3: Net-(U206A-+) -> unconnected-(U206A-+-Pad3)
- U206 pad 4: /Analog Audio/-V_OPA -> -6.5V
- U206 pad 5: Net-(U206B-+) -> unconnected-(U206B-+-Pad5)
- U206 pad 6: Net-(U206B--) -> unconnected-(U206B---Pad6)
- U206 pad 7: Net-(R227-Pad2) -> unconnected-(U206-Pad7)
- U206 pad 8: /Analog Audio/+V_OPA -> +6.5V
- U3 pad 5: FRAM_SDA -> /DSP/FRAM_SDA
- U3 pad 6: FRAM_SCL -> /DSP/FRAM_SCL
- U3 pad 7: FRAM_WP -> /DSP/FRAM_WP
- U3 pad 8: /Analog Audio/+3.3V -> +3.3V
- U4 pad 10: /Analog Audio/+V_OPA -> +6.5V
- U4 pad 6: /Analog Audio/-V_OPA -> -6.5V
- U5 pad 1: Net-(U5-CB) -> +5V_Clamp
- U5 pad 2: -7V -> Net-(U5-REF)
- U5 pad 3: Net-(U5-FB) -> GND
- Y1 pad 1: /Analog Audio/+3.3V -> +3.3V
- Y1 pad 3: Net-(U18-PH0) -> /DSP/AUDIOCLK
- Y1 pad 4: /Analog Audio/+3.3V -> +3.3V
Routing:
- net Net-(U18-PH0): track 2.12 -> 0.00 mm
- net /DSP/D+: track 1.98 -> 0.00 mm
- net /DSP/D-: track 1.97 -> 0.00 mm
- net UART0_RX: track 1.53 -> 0.00 mm
- net GND: track 0.63 -> 0.00 mm, vias 1 -> 0
Other:
- outline, holes or cut-outs redrawn
