File: ProjectY.kicad_pcb (KiCad board)
At the start: 6 copper layers, 100 x 85 mm, 266 parts, among them IC2 R7KA8P1KFLCAB#UC0, J15 009155002852006, J16 009155002852006, J17 Out, J2 Conn_ARM_JTAG_SWD_10, J3 9V, J5 IN_R, J6 IN_L, J7 Out, J9 USB_C_Receptacle_USB2.0_14P, K1 G6K-2, Q2 AO3401A, Q3 BC846, U1 W9825G6KH-6, U11 RT8293B, U12 USBLC6-2P6, U2 IS25LX512M-JHLE, U201 OPA1678, U202 OPA1678, U203 OPA1678, U204 OPA1678, U205 TAC5242, U206 OPA1678, U3 FM24CL64B, U4 TPS7A39, U5 TL431DBZ, U6 OPA1678, U8 TLV77325PDBVR, U9 TL431DBZ, Y1 ASDLJ-E-24.576MHZ-L-R-T, Y3 SG-5032CAN 24MHz

Commit message: progressed with SDRAM layout
Parts:
- removed C402, C403: 10uF, PCM_JLCPCB:C_0603
- removed D5: B5819W, Diode_SMD:D_SOD-123
- removed F1: 1A, Fuse:Fuse_0805_2012Metric
- removed Q2: AO3401A, Package_TO_SOT_SMD:SOT-23
- removed R29: 12k, Resistor_SMD:R_0603_1608Metric
- added C106: 6.8pF, PCM_JLCPCB:C_0402, F.Cu at (63.0, 125.9)
- added C107: 6.8pF, PCM_JLCPCB:C_0402, F.Cu at (65.9, 127.8)
- added C112: 4.7uF, PCM_JLCPCB:C_0402, F.Cu at (195.3, 162.1)
- added C113: 4.7uF, PCM_JLCPCB:C_0402, F.Cu at (199.6, 162.1)
- added C114: 4.7uF, PCM_JLCPCB:C_0402, F.Cu at (248.6, 61.1)
- added C115: 4.7uF, PCM_JLCPCB:C_0402, B.Cu at (183.1, 142.5)
- added C116: 4.7uF, PCM_JLCPCB:C_0402, F.Cu at (199.6, 147.6)
- added C117: 4.7uF, PCM_JLCPCB:C_0402, F.Cu at (210.8, 162.6)
- added C118: 4.7uF, PCM_JLCPCB:C_0402, F.Cu at (194.6, 147.6)
- added C119: 4.7uF, PCM_JLCPCB:C_0402, B.Cu at (184.6, 145.0)
- added C120: 4.7uF, PCM_JLCPCB:C_0402, B.Cu at (181.6, 146.0)
- added C51: 47uF, PCM_JLCPCB:C_1206, F.Cu at (74.1, 100.1)
- added C52: 100u, 60mR, Capacitor_Tantalum_SMD:CP_EIA-7343-31_Kemet-D, F.Cu at (237.4, 132.2)
- added C53: 1uF, PCM_JLCPCB:C_0603, F.Cu at (241.7, 118.2)
- added C54: 100nF, PCM_JLCPCB:C_0402, F.Cu at (236.2, 112.4)
- added C55: 47uF, PCM_JLCPCB:C_1206, F.Cu at (74.1, 95.3)
- added C56: 100nF, PCM_JLCPCB:C_0402, F.Cu at (80.5, 48.8)
- added C82: 10uF, PCM_JLCPCB:C_0805, F.Cu at (234.8, 137.8)
- added C83: 10uF, PCM_JLCPCB:C_0805, F.Cu at (234.8, 135.7)
- added C84: 100nF, PCM_JLCPCB:C_0402, F.Cu at (236.2, 111.5)
- added C85: 100nF, PCM_JLCPCB:C_0402, F.Cu at (236.2, 110.6)
- added C86: 100nF, PCM_JLCPCB:C_0402, F.Cu at (236.2, 109.7)
- added C87: 100nF, PCM_JLCPCB:C_0402, F.Cu at (75.0, 52.8)
- added C94: 47uF, PCM_JLCPCB:C_1206, F.Cu at (71.6, 95.4)
- added C95: 47uF, PCM_JLCPCB:C_1206, F.Cu at (69.1, 95.4)
- added C96: 47uF, PCM_JLCPCB:C_1206, F.Cu at (66.7, 95.4)
- added C97: 10nF, Capacitor_SMD:C_0603_1608Metric, F.Cu at (81.2, 109.6)
- added C98: 4.7nF, Capacitor_SMD:C_0603_1608Metric, F.Cu at (85.2, 112.0)
- added D7: B5819W, PCM_JLCPCB:D_SOD-123, F.Cu at (78.1, 109.9)
- added L6: 10u, Inductor_SMD:L_Sunlord_MWSA0518S, F.Cu at (72.7, 111.8)
- added L7: 10u, Inductor_SMD:L_Sunlord_MWSA0518S, F.Cu at (275.7, 101.0)
- added Q1: AO3401A, PCM_JLCPCB:Q_SOT-23, F.Cu at (71.8, 119.7)
- added R44: 12kΩ, PCM_JLCPCB:R_0402, F.Cu at (236.4, 120.2)
- added R45: 110kΩ, PCM_JLCPCB:R_0603, F.Cu at (241.7, 115.5)
- added R46: 8.2kΩ, PCM_JLCPCB:R_0603, F.Cu at (234.2, 120.4)
- added R47: 1.5kΩ, PCM_JLCPCB:R_0402, F.Cu at (232.3, 117.0)
- added R48: 510kΩ, PCM_JLCPCB:R_0402, F.Cu at (65.9, 129.6)
- added TP1: 3.3V, Thunderscope_Rev5.1:GEN_TP_PCB, F.Cu at (229.1, 155.6)
- added TP10: FB3, Thunderscope_Rev5.1:GEN_TP_PCB, F.Cu at (70.6, 134.2)
- added TP2: Bode, Thunderscope_Rev5.1:GEN_TP_PCB, F.Cu at (228.1, 20.8)
- added TP3: FB, Thunderscope_Rev5.1:GEN_TP_PCB, F.Cu at (231.2, 155.6)
- added TP4: 3.3V_GND, TestPoint:TestPoint_Pad_1.0x1.0mm, F.Cu at (226.6, 155.8)
- added TP5: Bode2, Thunderscope_Rev5.1:GEN_TP_PCB, F.Cu at (65.7, 131.8)
- added TP6: Bode3, Thunderscope_Rev5.1:GEN_TP_PCB, F.Cu at (65.7, 134.2)
- added TP7: 7V, Thunderscope_Rev5.1:GEN_TP_PCB, F.Cu at (68.2, 131.8)
- added TP8: -7V, Thunderscope_Rev5.1:GEN_TP_PCB, F.Cu at (68.5, 109.9)
- added TP9: FB2, Thunderscope_Rev5.1:GEN_TP_PCB, F.Cu at (70.6, 131.8)
- added U13: TPS259630, Package_SO:TI_SO-PowerPAD-8, F.Cu at (236.9, 116.9)
- added U17: TPS65131RGET, Package_DFN_QFN:VQFN-24-1EP_4x4mm_P0.5mm_EP2.5x2.5mm_ThermalVias, F.Cu at (81.0, 113.8)
- C1, C11, C2, C24, C36, C37, C38, C39, C40, C47, C5, C6, C60, C64, C65, C68, C69, C7, C71, C72, C73, C74, C75, C8, C9: moved to B.Cu
- C10: value 10uF -> 4.7uF
- C25, C26: value 10u -> 10uF; footprint Capacitor_SMD:C_1206_3216Metric -> PCM_JLCPCB:C_0402
- C27: value 100n -> 100nF; footprint Capacitor_SMD:C_0603_1608Metric -> PCM_JLCPCB:C_0402
- C28: value 10n -> 10uF; footprint Capacitor_SMD:C_0603_1608Metric -> PCM_JLCPCB:C_0402
- C29: value 6p8 -> 10uF; footprint Capacitor_SMD:C_0603_1608Metric -> PCM_JLCPCB:C_0402
- C30: value 8p2 -> 4.7uF; footprint Capacitor_SMD:C_0603_1608Metric -> PCM_JLCPCB:C_0402; moved to B.Cu
- C31: value 220n -> 220nF; footprint Capacitor_SMD:C_0603_1608Metric -> PCM_JLCPCB:C_0402
- C32, C33: value 22u -> 47uF; footprint Capacitor_SMD:C_0805_2012Metric -> PCM_JLCPCB:C_1206
- C34: value 4n7 -> 47uF; footprint Capacitor_SMD:C_0603_1608Metric -> PCM_JLCPCB:C_1206
- D4: footprint Diode_SMD:D_SOD-123 -> PCM_JLCPCB:D_SOD-123
- L3: footprint Inductor_SMD:L_12x12mm_H8mm -> User:WE-PD_1030P
- L4: value 1uH -> 22uH; footprint Inductor_SMD:L_1008_2520Metric -> Inductor_SMD:L_7.3x7.3_H3.5
- R12: value 0Ω -> 1
- R23: value 100 -> 47Ω; footprint Resistor_SMD:R_0603_1608Metric -> PCM_JLCPCB:R_0402
- R24: value 1M -> 100Ω; footprint Resistor_SMD:R_0603_1608Metric -> PCM_JLCPCB:R_0603
- R25: value 110k -> 47Ω; footprint Resistor_SMD:R_0603_1608Metric -> PCM_JLCPCB:R_0402
- R26: value 100k -> 100kΩ; footprint Resistor_SMD:R_0603_1608Metric -> PCM_JLCPCB:R_0402
- R27: value 1M -> 510kΩ; footprint Resistor_SMD:R_0603_1608Metric -> PCM_JLCPCB:R_0402
- R28: value 12k -> 100kΩ; footprint Resistor_SMD:R_0603_1608Metric -> PCM_JLCPCB:R_0402
- moved C36 177.7 mm to (178.8, 165.4)
- moved C37 177.0 mm to (178.8, 166.3)
- moved C2 173.0 mm to (178.2, 156.0), turned to 180 degrees
- moved C1 172.1 mm to (178.2, 152.7), turned to 180 degrees
- moved C38 171.2 mm to (174.1, 164.6), turned to 180 degrees
- moved C40 169.7 mm to (186.5, 151.5), turned to 180 degrees
- moved C39 169.4 mm to (174.2, 163.7), turned to 180 degrees
- moved C71 169.0 mm to (170.9, 164.7)
- moved C74 166.7 mm to (181.6, 156.0), turned to 180 degrees
- moved C72 166.3 mm to (170.9, 162.8)
- moved C81 165.4 mm to (234.8, 139.9), turned to 180 degrees
- moved C47 165.3 mm to (172.1, 159.3)
- moved C6 165.2 mm to (167.3, 160.1), turned to 180 degrees
- moved C5 164.5 mm to (175.4, 148.0)
- moved C68 164.2 mm to (181.6, 154.3), turned to 180 degrees
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Connections:
- net Net-(IC2A-VCL0) renamed /PSU/MCU_DCDC_OUT
- C19 pad 1: Net-(C19-Pad1) -> +3.3V
- C20 pad 1: Net-(C19-Pad1) -> +3.3V
- C21 pad 1: Net-(C19-Pad1) -> +3.3V
- C22 pad 1: Net-(C19-Pad1) -> +3.3V
- C25 pad 1: +5V -> Net-(C25-Pad1)
- C26 pad 1: Net-(Q2-D) -> Net-(Q1-D)
- C27 pad 1: Net-(IC1-ENN) -> Net-(U17-ENN)
- C28 pad 1: Net-(IC1-CP) -> Net-(Q1-D)
- C29 pad 1: +12V -> Net-(Q1-D)
- C29 pad 2: Net-(IC1-FBP) -> GND
- C30 pad 1: Net-(IC1-FBN) -> +3.3V
- C30 pad 2: -12V -> GND
- C31 pad 1: Net-(IC1-VREF) -> GND
- C31 pad 2: GND -> Net-(U17-VREF)
- C32 pad 1: -12V -> GND
- C32 pad 2: GND -> -7V
- C33 pad 1: +12V -> GND
- C33 pad 2: GND -> -7V
- C34 pad 1: Net-(IC1-CN) -> GND
- C34 pad 2: GND -> -7V
- D4 pad 1: +12V -> Net-(U17-OUT_N)
- D4 pad 2: Net-(D4-A) -> -7V
- IC2 pad N8: unconnected-(IC2A-AVCC0-PadN8) -> +2.5V
- IC2 pad P4: unconnected-(IC2A-AVCC_MIPI-PadP4) -> +3.3V
- IC2 pad R8: unconnected-(IC2A-VREFH-PadR8) -> +2.5V
- IC2 pad R9: unconnected-(IC2A-VREFH0-PadR9) -> +2.5V
- L3 pad 2: Net-(C19-Pad1) -> +3.3V
- R2 pad 2: Net-(C19-Pad1) -> +3.3V
- R23 pad 1: Net-(IC1-ENN) -> Net-(C106-Pad1)
- R23 pad 2: +5V -> +7V
- R24 pad 1: Net-(IC1-FBP) -> Net-(C25-Pad1)
- R24 pad 2: +12V -> Net-(U17-ENN)
- R25 pad 1: GND -> -7V
- R25 pad 2: Net-(IC1-FBP) -> Net-(C107-Pad2)
- R26 pad 1: Net-(IC1-FBN) -> Net-(U17-FBP)
- R26 pad 2: Net-(IC1-VREF) -> GND
- R27 pad 1: -12V -> Net-(C107-Pad2)
- R27 pad 2: Net-(IC1-FBN) -> Net-(U17-FBN)
- R28 pad 1: GND -> Net-(U17-VREF)
- R28 pad 2: -12V -> Net-(U17-FBN)
- U1 pad 10: /DSP/RAM_D5 -> /DSP/RAM_D4
- U1 pad 4: /DSP/RAM_D1 -> /DSP/RAM_D2
- U1 pad 45: /DSP/RAM_D10 -> /DSP/RAM_D12
- U1 pad 47: /DSP/RAM_D11 -> /DSP/RAM_D14
- U1 pad 48: /DSP/RAM_D12 -> /DSP/RAM_D13
- U1 pad 5: /DSP/RAM_D2 -> /DSP/RAM_D1
- U1 pad 50: /DSP/RAM_D13 -> /DSP/RAM_D15
- U1 pad 51: /DSP/RAM_D14 -> /DSP/RAM_D10
- U1 pad 53: /DSP/RAM_D15 -> /DSP/RAM_D11
- U1 pad 8: /DSP/RAM_D4 -> /DSP/RAM_D5
- U6 pad 4: (no net) -> -6.5V
- U6 pad 8: (no net) -> +6.5V
Routing:
- net /DSP/RAM_A3: track 0.00 -> 29.2 mm, vias 0 -> 2
- net /DSP/RAM_BA1: track 0.00 -> 28.7 mm, vias 0 -> 3
- net /DSP/RAM_A1: track 0.00 -> 28.2 mm, vias 0 -> 2
- net /DSP/RAM_A2: track 0.00 -> 28.1 mm
- net /DSP/RAM_A4: track 0.00 -> 28.0 mm
- net /DSP/RAM_A10: track 0.00 -> 27.6 mm
- net /DSP/RAM_A5: track 0.00 -> 27.4 mm
- net /DSP/RAM_CKE: track 0.00 -> 27.2 mm, vias 0 -> 2
- net /DSP/RAM_A6: track 0.00 -> 26.6 mm, vias 0 -> 2
- net /DSP/RAM_A7: track 0.00 -> 26.4 mm, vias 0 -> 2
- net /DSP/RAM_A0: track 0.00 -> 25.5 mm
- net /DSP/RAM_BA0: track 0.00 -> 24.9 mm, vias 0 -> 2
- net /DSP/RAM_A9: track 0.00 -> 23.8 mm, vias 0 -> 2
- net /DSP/RAM_A11: track 0.00 -> 23.5 mm, vias 0 -> 2
- net /DSP/RAM_A8: track 0.00 -> 23.3 mm
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- added copper zone on In4.Cu, net +3.3V
- added copper zone on In4.Cu, net /PSU/MCU_DCDC_OUT
- added copper zone on F.Cu, net Net-(IC2A-VLO_1)

Commit message: layout progress
Parts:
- removed C100, C101, C102, C103, C104, C105, C90, C91, C92, C93, C99: 100nF, PCM_JLCPCB:C_0402
- removed C12, C13: 47uF, PCM_JLCPCB:C_1206
- removed C46: 4.7uF, PCM_JLCPCB:C_0402
- removed D201, D202, D203, D204: BAV99, Package_TO_SOT_SMD:SOT-23
- removed J15, J16: 009155002852006, User:KYO_009155002852006
- removed R10, R19, R20, R21, R3, R6, R74, R78, R84, R85, R86, R87, R92, R93, R94, R95, R96, R97: 10kΩ, PCM_JLCPCB:R_0402
- removed R30, R37, R38, R4, R41, R42: 1kΩ, PCM_JLCPCB:R_0402
- removed U5, U9: TL431DBZ, Package_TO_SOT_SMD:SOT-23
- removed U8: TLV77325PDBVR, Package_TO_SOT_SMD:SOT-23-5
- added C58: 100u, 60mR, Capacitor_Tantalum_SMD:CP_EIA-7343-31_Kemet-D, F.Cu at (185.6, 133.3)
- added D10: ESD401, PCM_JLCPCB:D_DFN1006-2L, B.Cu at (183.1, 106.8)
- added D11: H5VL10B, PCM_JLCPCB:D_DFN1006-2L, F.Cu at (202.0, 141.3)
- added D12: H5VL10B, PCM_JLCPCB:D_DFN1006-2L, F.Cu at (198.8, 141.3)
- added D13: H5VL10B, PCM_JLCPCB:D_DFN1006-2L, F.Cu at (200.4, 141.3)
- added D14: H5VL10B, PCM_JLCPCB:D_DFN1006-2L, F.Cu at (197.2, 141.3)
- added D15: H5VL10B, PCM_JLCPCB:D_DFN1006-2L, F.Cu at (195.6, 141.3)
- added D16: H5VL10B, PCM_JLCPCB:D_DFN1006-2L, F.Cu at (193.7, 148.4)
- added D17: H5VL10B, PCM_JLCPCB:D_DFN1006-2L, F.Cu at (202.7, 154.9)
- added D18: H5VL10B, PCM_JLCPCB:D_DFN1006-2L, F.Cu at (199.4, 154.7)
- added D19: H5VL10B, PCM_JLCPCB:D_DFN1006-2L, F.Cu at (205.7, 154.9)
- added D20: 1N4148W, PCM_JLCPCB:D_SOD-123, F.Cu at (183.7, 124.0)
- added D5: ESD401, PCM_JLCPCB:D_DFN1006-2L, B.Cu at (165.0, 113.2)
- added D8: ESD401, PCM_JLCPCB:D_DFN1006-2L, B.Cu at (199.8, 113.1)
- added D9: ESD401, PCM_JLCPCB:D_DFN1006-2L, B.Cu at (183.1, 114.2)
- added FB4: ?, Inductor_SMD:L_0805_2012Metric, F.Cu at (192.8, 131.8)
- added H1: MountingHole, MountingHole:MountingHole_2.7mm_M2.5, F.Cu at (238.9, 160.9)
- added H2: MountingHole, MountingHole:MountingHole_2.7mm_M2.5, F.Cu at (146.9, 160.9)
- added H3: MountingHole, MountingHole:MountingHole_2.7mm_M2.5, F.Cu at (192.9, 125.9)
- added J1: UI Board Connector, Connector_SMD_Wurth:J_Wurth_WR-MM_690367280676, F.Cu at (202.9, 159.7)
- added NT1: NetTie_2, NetTie:NetTie-2_SMD_Pad0.5mm, F.Cu at (155.7, 122.3)
- added R29: 47Ω, PCM_JLCPCB:R_0402, F.Cu at (211.0, 124.4)
- added R57: 0, PCM_JLCPCB:R_0402, F.Cu at (190.6, 131.8)
- added TP11: +6.5V, TestPoint:TestPoint_Pad_1.0x1.0mm, B.Cu at (151.9, 162.1)
- added TP12: -6.5V, TestPoint:TestPoint_Pad_1.0x1.0mm, B.Cu at (151.8, 154.9)
- added U10: ISOUSB111DWXR, User:SOIC16_DW_TEX-L, F.Cu at (224.6, 111.6)
- C10, C219, C220, C35, C401, C41, C42, C43, C44, C45, C50, C57, C63, C70, C76, C77, C78, C81, R36, R39, R40, R43, R47, TP10, TP5, TP6, TP7, TP9: moved to B.Cu
- C115, C119, C120, C47, C60, C64, C65, C71, C72: moved to F.Cu
- C62: value 10uF -> 4.7uF
- C88: value 100nF -> 1uF
- C89: value 100nF -> 10uF
- D2, D3: value BAV99 -> ESD401; footprint Package_TO_SOT_SMD:SOT-23 -> PCM_JLCPCB:D_DFN1006-2L; moved to B.Cu
- J2: footprint Connector_PinHeader_2.54mm:PinHeader_1x02_P2.54mm_Vertical -> Connector_PinHeader_1.27mm:PinHeader_2x05_P1.27mm_Vertical_SMD
- R226, R228: footprint Resistor_SMD:R_0402_1005Metric -> PCM_JLCPCB:R_0402
- U17: footprint Package_DFN_QFN:VQFN-24-1EP_4x4mm_P0.5mm_EP2.5x2.5mm_ThermalVias -> User:VQFN-24-1EP_4x4mm_P0.5mm_EP2.5x2.5mm_ThermalVias
- moved C44 191.3 mm to (220.4, 134.0)
- moved C35 187.5 mm to (217.3, 126.7), turned to 90 degrees
- moved C45 185.7 mm to (218.1, 128.6), turned to -90 degrees
- moved C41 179.4 mm to (212.6, 128.9), turned to 90 degrees
- moved C43 178.6 mm to (212.6, 130.8), turned to -90 degrees
- moved C42 177.8 mm to (211.8, 128.9), turned to 90 degrees
- moved C70 175.3 mm to (211.8, 130.8), turned to -90 degrees
- moved R36 159.1 mm to (196.4, 116.8)
- moved R35 142.1 mm to (209.8, 122.4), turned to 90 degrees
- moved R9 135.1 mm to (168.3, 130.7), turned to 90 degrees
- moved TP2 135.0 mm to (231.2, 155.7)
- moved R31 134.1 mm to (214.1, 125.0), turned to 180 degrees
- moved C209 131.5 mm to (168.3, 128.8), turned to 90 degrees
- moved R34 130.8 mm to (214.1, 120.7), turned to 180 degrees
- moved R17 126.3 mm to (175.0, 131.1), turned to 180 degrees
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Connections:
- C25 pad 1: Net-(C25-Pad1) -> +3.3V
- C62 pad 1: +2.5V -> +3.3V
- C88 pad 1: Net-(C88-Pad1) -> /DSP/VBUS
- C88 pad 2: GND -> ISO_GND
- C89 pad 1: Net-(C89-Pad1) -> Net-(Q1-D)
- D2 pad 1: -5V_Clamp -> /Analog Audio/IN_L
- D2 pad 2: +5V_Clamp -> GND
- D3 pad 1: -5V_Clamp -> /Analog Audio/Line_Output_R-
- D3 pad 2: +5V_Clamp -> GND
- IC2 pad A15: unconnected-(IC2D-P206-PadA15) -> /Analog Audio/~{Analog_Dry}
- IC2 pad D14: unconnected-(IC2D-P707-PadD14) -> Net-(IC2D-UART_TXD1)
- IC2 pad D15: unconnected-(IC2D-P706-PadD15) -> /DSP/UART_RX
- IC2 pad M8: /DSP/Switch_1A -> unconnected-(IC2D-ADC1_9-PadM8)
- IC2 pad M9: /DSP/Footswitch_2 -> unconnected-(IC2D-ADC1_7-PadM9)
- IC2 pad N10: /DSP/Potentiometer_6 -> unconnected-(IC2D-ADC0_5-PadN10)
- IC2 pad N11: /DSP/Potentiometer_2 -> unconnected-(IC2D-ADC0_1-PadN11)
- IC2 pad N8: +2.5V -> +3.3V
- IC2 pad P10: /DSP/Switch_1B -> unconnected-(IC2D-ADC1_6-PadP10)
- IC2 pad P11: /DSP/Potentiometer_3 -> unconnected-(IC2D-ADC0_2-PadP11)
- IC2 pad P12: /DSP/Potentiometer_4 -> unconnected-(IC2D-ADC0_3-PadP12)
- IC2 pad P7: /DSP/Switch_2B -> unconnected-(IC2D-ADC1_15-PadP7)
- IC2 pad R10: /DSP/Footswitch_1 -> unconnected-(IC2D-ADC1_8-PadR10)
- IC2 pad R11: /DSP/Potentiometer_5 -> unconnected-(IC2D-ADC0_4-PadR11)
- IC2 pad R12: /DSP/Potentiometer_1 -> unconnected-(IC2D-ADC0_0-PadR12)
- IC2 pad R7: /DSP/Switch_2A -> unconnected-(IC2D-ADC0_14-PadR7)
- IC2 pad R8: +2.5V -> +3.3V
- IC2 pad R9: +2.5V -> +3.3V
- J5 pad R: GND -> AGND
- J5 pad RN: GND -> AGND
- J5 pad S: GND -> AGND
- J5 pad SN: GND -> AGND
- J5 pad TN: GND -> /Analog Audio/IN_L
- J6 pad R: GND -> AGND
- J6 pad RN: GND -> AGND
- J6 pad S: GND -> AGND
- J6 pad SN: GND -> AGND
- J6 pad TN: GND -> AGND
- K1 pad 4: GND -> AGND
- K1 pad 5: GND -> AGND
- R203 pad 2: GND -> AGND
- R204 pad 2: GND -> AGND
- R207 pad 2: GND -> AGND
- R210 pad 2: GND -> AGND
- R214 pad 2: GND -> AGND
- R216 pad 2: GND -> AGND
- R223 pad 1: GND -> AGND
- R226 pad 1: GND -> AGND
- R24 pad 1: Net-(C25-Pad1) -> +3.3V
- R39 pad 1: GND -> AGND
- R43 pad 1: GND -> AGND
- R55 pad 6: /DSP/FLASH_~{INT} -> /DSP/FLASH_~{RST}
- R55 pad 8: /DSP/FLASH_~{RST} -> /DSP/FLASH_~{INT}
- U12 pad 1: Net-(U10-UD-) -> /DSP/UD+
- U12 pad 3: Net-(U10-UD+) -> /DSP/UD-
- U12 pad 4: /DSP/D+ -> /DSP/D-
- U12 pad 6: /DSP/D- -> /DSP/D+
- U17 pad 20: unconnected-(U17-NC-Pad12) -> unconnected-(U17-NC_2-Pad20)
- U206 pad 3: GND -> AGND
- U206 pad 5: GND -> AGND
Routing:
- net AGND: track 0.00 -> 77.5 mm
- net DAC_R-: track 0.00 -> 48.2 mm
- net DAC_R+: track 0.00 -> 37.9 mm
- net Net-(U11-VIN): track 0.00 -> 23.5 mm, vias 0 -> 1
- net GND: track 23.1 -> 42.9 mm, vias 45 -> 90
- net DAC_L+: track 0.00 -> 18.4 mm
- net Net-(D1-Pad1): track 0.00 -> 15.5 mm
- net Net-(U11-SW): track 0.00 -> 13.6 mm, vias 0 -> 2
- net Net-(U13-OUT): track 0.00 -> 13.0 mm
- net Net-(C232-Pad2): track 0.00 -> 12.3 mm
- net /Analog Audio/IN_L: track 0.00 -> 11.0 mm
- net DAC_L-: track 0.00 -> 10.5 mm
- net Net-(K1-Pad3): track 0.00 -> 9.39 mm
- net Net-(U6A--): track 0.00 -> 8.01 mm
- net +6.5V: track 0.00 -> 7.90 mm, vias 0 -> 5
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- added copper zone on F.Cu, net +3.3V
- added copper zone on F.Cu, net Net-(U11-VIN)
- added copper zone on F.Cu, net Net-(U13-IN)
Other:
- board size 100 x 85 mm -> 100 x 70 mm

Commit message: progressed with the layout
Parts:
- removed C231, C232, C235, C236: 47uF, Capacitor_SMD:C_Elec_6.3x7.7
- removed FB4: ?, Inductor_SMD:L_0805_2012Metric
- removed R57: 0, PCM_JLCPCB:R_0402
- removed TP10: FB3, Thunderscope_Rev5.1:GEN_TP_PCB
- removed TP5: Bode2, Thunderscope_Rev5.1:GEN_TP_PCB
- removed TP6: Bode3, Thunderscope_Rev5.1:GEN_TP_PCB
- removed TP7: 7V, Thunderscope_Rev5.1:GEN_TP_PCB
- removed TP8: -7V, Thunderscope_Rev5.1:GEN_TP_PCB
- removed TP9: FB2, Thunderscope_Rev5.1:GEN_TP_PCB
- added C12: 10uF, PCM_JLCPCB:C_0402, F.Cu at (181.5, 152.4)
- added C13: 10uF, PCM_JLCPCB:C_0402, F.Cu at (182.4, 152.4)
- added C46: 10uF, PCM_JLCPCB:C_0402, F.Cu at (183.3, 152.4)
- added C61: 4.7uF, PCM_JLCPCB:C_0402, B.Cu at (255.0, 138.9)
- added C90: 4.7uF, PCM_JLCPCB:C_0402, B.Cu at (215.9, 130.8)
- added C91: 4.7uF, PCM_JLCPCB:C_0402, B.Cu at (215.1, 130.8)
- C107, C31, C62, C64, C65, C71, C72, C97, C98, R24, R25, R27, R28: moved to B.Cu
- C58: value 100u, 60mR -> 4.7uF; footprint Capacitor_Tantalum_SMD:CP_EIA-7343-31_Kemet-D -> PCM_JLCPCB:C_0402
- moved C58 86.4 mm to (270.8, 118.6), turned to 0 degrees
- moved C71 71.0 mm to (276.2, 139.9), turned to -90 degrees
- moved C69 69.4 mm to (285.6, 120.8), turned to -90 degrees
- moved C9 61.6 mm to (274.7, 143.7)
- moved C2 60.5 mm to (274.7, 134.4), turned to 180 degrees
- moved C8 59.8 mm to (274.7, 141.8), turned to 180 degrees
- moved C1 56.9 mm to (274.7, 132.6), turned to 180 degrees
- moved C65 51.6 mm to (255.8, 138.9), turned to -90 degrees
- moved C47 50.7 mm to (253.0, 106.1)
- moved C60 50.7 mm to (253.9, 106.1)
- moved C57 48.9 mm to (261.6, 136.0), turned to 180 degrees
- moved C72 48.4 mm to (254.2, 138.9), turned to -90 degrees
- moved C38 41.0 mm to (256.4, 129.6), turned to 180 degrees
- moved C75 39.0 mm to (256.6, 139.1), turned to -90 degrees
- moved C30 37.7 mm to (257.9, 123.9), turned to 0 degrees
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Connections:
- C241 pad 1: /Analog Audio/3.3V_AVDD -> +3.3V
- C58 pad 1: Net-(C58-Pad1) -> /PSU/MCU_DCDC_OUT
- D20 pad 1: /Analog Audio/3.3V_AVDD -> +3.3V
- K1 pad 1: /Analog Audio/3.3V_AVDD -> +3.3V
- R221 pad 1: Net-(C231-Pad2) -> DAC_R-
- R222 pad 1: Net-(C232-Pad2) -> DAC_R+
- R224 pad 1: Net-(C235-Pad2) -> DAC_L-
- R225 pad 1: Net-(C236-Pad2) -> DAC_L+
- U202 pad 3: GND -> AGND
- U202 pad 5: GND -> AGND
- U205 pad 23: /Analog Audio/3.3V_AVDD -> +3.3V
- U205 pad 7: /Analog Audio/3.3V_AVDD -> +3.3V
- U205 pad 8: /Analog Audio/3.3V_AVDD -> +3.3V
Routing:
- net AGND: track 77.5 -> 157.7 mm, vias 0 -> 15
- net /DSP/UART_TX: track 0.00 -> 47.2 mm
- net /DSP/UART_RX: track 0.00 -> 46.9 mm
- net /Analog Audio/I2S_RX: track 0.00 -> 35.9 mm, vias 0 -> 2
- net /Analog Audio/I2S_TX: track 0.00 -> 35.3 mm, vias 0 -> 2
- net /Analog Audio/Analog_Dry_In_R: track 0.00 -> 35.2 mm
- net /Analog Audio/I2S_WS: track 0.00 -> 34.2 mm, vias 0 -> 3
- net /Analog Audio/Effect_Signal_R: track 1.99 -> 35.5 mm, vias 0 -> 2
- net Net-(C204-Pad1): track 2.06 -> 31.3 mm
- net /Analog Audio/I2S_CK: track 0.00 -> 28.6 mm, vias 0 -> 2
- net /Analog Audio/IN_L: track 11.0 -> 39.6 mm
- net /Analog Audio/Analog_Dry_In_L: track 2.54 -> 29.7 mm
- net ADC_R+: track 0.00 -> 21.2 mm
- net /Analog Audio/Effect_Signal_L: track 1.49 -> 22.4 mm, vias 0 -> 2
- net Net-(C204-Pad2): track 0.00 -> 19.5 mm
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- added copper zone on F.Cu, net +6.5V
- added copper zone on In3.Cu, net +6.5V
- added copper zone on F.Cu, net -6.5V
- added copper zone on In4.Cu, net -6.5V
- added copper zone on F.Cu, net /PSU/MCU_DCDC_OUT

Commit message: DCDC upgraded
Parts:
- removed C69, C71: 4.7uF, PCM_JLCPCB:C_0402
- added TP10: FB3, Thunderscope_Rev5.1:GEN_TP_PCB, F.Cu at (147.2, 184.6)
- added TP5: Bode2, Thunderscope_Rev5.1:GEN_TP_PCB, F.Cu at (142.3, 182.2)
- added TP6: Bode3, Thunderscope_Rev5.1:GEN_TP_PCB, F.Cu at (142.3, 184.6)
- added TP7: 7V, Thunderscope_Rev5.1:GEN_TP_PCB, F.Cu at (144.7, 182.2)
- added TP8: -7V, Thunderscope_Rev5.1:GEN_TP_PCB, F.Cu at (144.7, 184.6)
- added TP9: FB2, Thunderscope_Rev5.1:GEN_TP_PCB, F.Cu at (147.2, 182.2)
- C106, R23, R26, R48: moved to B.Cu
- C61, C65, C72, C75: moved to F.Cu
- moved C47 53.0 mm to (205.2, 128.8)
- moved C60 53.0 mm to (206.1, 128.8)
- moved C75 50.8 mm to (206.9, 128.8), turned to 90 degrees
- moved C65 49.1 mm to (207.7, 128.8), turned to 90 degrees
- moved C61 47.5 mm to (208.6, 128.8), turned to 90 degrees
- moved C72 45.9 mm to (209.4, 128.8), turned to 90 degrees
- moved R26 8.67 mm to (180.7, 158.0), turned to -90 degrees
- moved C106 7.28 mm to (179.8, 158.0), turned to 90 degrees
- moved R48 6.31 mm to (178.9, 158.0), turned to -90 degrees
- moved R23 4.93 mm to (179.4, 159.3), turned to 180 degrees
- moved R25 3.06 mm to (174.2, 156.5)
- moved C51 0.90 mm to (171.1, 159.9)
- moved C34 0.90 mm to (168.7, 159.9)
- moved L7 0.90 mm to (170.5, 154.2), turned to -90 degrees
- moved C97 0.60 mm to (177.7, 158.6)
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Routing:
- net Net-(Q1-G): track 0.00 -> 14.6 mm
- net GND: track 51.3 -> 64.0 mm, vias 133 -> 178
- net Net-(U17-ENN): track 2.63 -> 8.30 mm, vias 0 -> 2
- net Net-(U17-FBN): track 0.00 -> 2.84 mm, vias 0 -> 1
- net Net-(U17-FBP): track 0.00 -> 2.81 mm, vias 0 -> 1
- net +3.3V: track 28.5 -> 31.1 mm, vias 48 -> 69
- net Net-(U17-VREF): track 0.00 -> 2.09 mm, vias 0 -> 1
- net Net-(U205-VREF): track 0.00 -> 1.98 mm
- net Net-(C107-Pad2): track 0.00 -> 1.89 mm
- net Net-(C106-Pad1): track 0.00 -> 1.79 mm
- net Net-(U17-CN): track 0.00 -> 1.69 mm, vias 0 -> 1
- net Net-(U17-CP): track 0.00 -> 1.28 mm, vias 0 -> 1
- net Net-(U205-DREG): track 0.00 -> 1.19 mm
- net -7V: track 0.00 -> 0.32 mm, vias 0 -> 1
- net +7V: vias 0 -> 1
- added copper zone on F.Cu, net +7V
- added copper zone on F.Cu, net -7V
- added copper zone on B.Cu, net GND
- added copper zone on F.Cu, net GND
- added copper zone on F.Cu, net Net-(Q1-D)
- added copper zone on F.Cu, net Net-(U17-INP)
- added copper zone on F.Cu, net Net-(U17-OUT_N)
