File: PSU.kicad_sch (KiCad schematic)
At the start: 126 parts, among them IC2 R7KA8P1KFLCAB#UC0, J3 9V, U11 RT8293B, U13 TPS259630, U17 TPS65131RGET, U4 TPS7A39

Commit message: signal integrity related fixes
Parts:
- added TP13: GND, TestPoint:TestPoint_Pad_1.0x1.0mm, symbol Connector:TestPoint
Connections:
- net GND: now also TP13.1
Changed lines of the file:
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@@
 	)
 	(junction
+		(at 138.43 262.89)
+		(diameter 0)
+		(color 0 0 0 0)
+	)
+	(junction
 		(at 233.68 29.21)
 		(diameter 0)
@@
 	(wire
 		(pts
-			(xy 127 262.89) (xy 143.51 262.89)
+			(xy 127 262.89) (xy 138.43 262.89)
 		)
 		(stroke
@@
 	(wire
 		(pts
+			(xy 138.43 262.89) (xy 143.51 262.89)
+		)
+		(stroke
+			(width 0)
+			(type default)
+		)
+	)
+	(wire
+		(pts
 			(xy 161.29 29.21) (xy 165.1 29.21)
 		)
@@
 					(unit 1)
 				)
+			)
+		)
+	)
+	(symbol
+		(lib_id "Connector:TestPoint")
+		(at 138.43 262.89 0)
+		(unit 1)
+		(exclude_from_sim no)
+		(in_bom yes)
+		(on_board yes)
+		(dnp no)
+		(fields_autoplaced yes)
+		(property "Reference" "TP13"
+			(at 140.97 258.3179 0)
+			(effects
+				(font
+					(size 1.27 1.27)
+				)
+				(justify left)
+			)
+		)
+		(property "Value" "GND"
+			(at 140.97 260.8579 0)
+			(effects
+				(font
+					(size 1.27 1.27)
+				)
+				(justify left)
+			)
+		)
+		(property "Footprint" "TestPoint:TestPoint_Pad_1.0x1.0mm"
+			(at 143.51 262.89 0)
+			(effects
+				(font
+					(size 1.27 1.27)
+				)
+				(hide yes)
+			)
+		)
+		(property "Datasheet" "~"
+			(at 143.51 262.89 0)
+			(effects
+				(font
+					(size 1.27 1.27)
+				)
+				(hide yes)
+			)
+		)
+		(property "Description" "test point"
+			(at 138.43 262.89 0)
+			(effects
+				(font
+					(size 1.27 1.27)
+				)
+				(hide yes)
+			)
+		)
+		(pin "1"
+		)
+		(instances
+			(project "ProjectY"
+				(path "/6b669608-d244-47fa-b233-c11102b937f7/f81f6974-b487-4052-a7d6-483d2ffe3d9e"
+					(reference "TP13")
+					(unit 1)
+				)
